File: PCB/quartz58.kicad_sch (KiCad schematic)
At the start: 60 parts, among them SW1 Switch, U1 Arduino_Pro_Micro

Commit message: small progress on left
Parts:
- removed SW1: Switch, symbol ScottoKeebs:Placeholder_Switch
- added D30: LED_SK6812MINI, ScottoKeebs_Components:LED_SK6812MINI, symbol ScottoKeebs:LED_SK6812MINI
- added Display1: nice!view, nice_view:nice_view, symbol nice_view:nice!view
- added J1: OLED_128x32, ScottoKeebs_Components:OLED_128x32, symbol ScottoKeebs:OLED_128x32
- added U2: ~, ScottoKeebs_Components:Encoder_Ano, symbol ScottoKeebs:Encoder_Ano
- added U3: TRRS, ScottoKeebs_Components:TRRS_PJ-320A, symbol ScottoKeebs:Placeholder_TRRS
Connections:
- net ROW5 is gone; now on net ROW2: U1.15 (14/PB3)
- net COL0: now also U1.1 (TX0/PD3)
- net COL1: now also U1.2 (RX1/PD2)
- net COL2: now also U1.7 (4/PD4)
- net COL3: now also U1.8 (5/PC6)
- net COL4: now also U1.9 (6/PD7)
- net ROW0: now also U1.17 (A0/PF7); no longer U1.20 (A3/PF4)
- net ROW1: now also U1.16 (15/PB1); no longer U1.19 (A2/PF5)
- net ROW2: no longer U1.18 (A1/PF6)
- net ROW3: now also U1.14 (16/PB2); no longer U1.17 (A0/PF7)
- net ROW4: now also U1.13 (10/PB6); no longer U1.16 (15/PB1)
- net COL5: now reaches S12.1, S23.1, S24.1, S29.1, S6.1
- net COL5: now also U1.10 (7/PE6)
- net VCC: now reaches U1.21 (VCC)
- net VCC: now also Display1.3 (VCC), J1.2 (VCC), U3.2 (TIP)
- net GND: now reaches U1.4 (GND)
- net GND: now also Display1.4 (GND), J1.1 (GND), U3.1 (SLEEVE)
- net SDA: now reaches U1.5 (2/PD1)
- net SDA: now also Display1.1 (MOSI), J1.4 (SDA)
- net SCL: now reaches U1.6 (3/PD0)
- net SCL: now also Display1.2 (SCK), J1.3 (SCL)
- new net CS: Display1.5 (CS), U1.20 (A3/PF4)
- new net RGB: D30.4 (DIN), U1.19 (A2/PF5)
Other:
- note added: "ANO ENCODER"
- note added: "Display"
- note added: "LEFT SIDE"
- note added: "RGB"
- moved on the sheet: D1, D10, D11, D12, D13, D14, D15, D16, D17, D18, D19, D2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

Commit message: easy stuff on pcb done
Parts:
- removed U1: Arduino_Pro_Micro, ScottoKeebs_MCU:Arduino_Pro_Micro, symbol ScottoKeebs:MCU_Arduino_Pro_Micro
- removed U2: ~, ScottoKeebs_Components:Encoder_Ano, symbol ScottoKeebs:Encoder_Ano
- removed U3: TRRS, ScottoKeebs_Components:TRRS_PJ-320A, symbol ScottoKeebs:Placeholder_TRRS
- added BT1: Battery_Cell, symbol Device:Battery_Cell
- added D100, D101, D102, D103, D104, D105, D106, D107, D108, D109, D110, D111, D112, D113, D114, D115, D116, D117, D118, D119, D120, D121, D31, D32, D33, D34, D35, D36, D37, D38, D39, D40, D41, D42, D43, D44, D45, D46, D47, D48, D49, D50, D51, D52, D53, D54, D55, D56, D57, D58, D93, D94, D95, D96, D97, D98, D99: LED_SK6812MINI, ScottoKeebs_Components:LED_SK6812MINI, symbol ScottoKeebs:LED_SK6812MINI
- added D59, D60, D61, D62, D63, D64, D65, D66, D67, D68, D69, D70, D71, D72, D73, D74, D75, D76, D77, D78, D79, D80, D81, D82, D83, D84, D85, D86, D87, D88, D89, D90, D91, D92: Diode, symbol ScottoKeebs:Placeholder_Diode
- added Display2: nice!view, nice_view:nice_view, symbol nice_view:nice!view
- added J2: OLED_128x32, ScottoKeebs_Components:OLED_128x32, symbol ScottoKeebs:OLED_128x32
- added S30, S31, S32, S33, S34, S35, S36, S37, S38, S39, S40, S41, S42, S43, S44, S45, S46, S47, S48, S49, S50, S51, S52, S53, S54, S55, S56, S57, S58, S59, S60, S61, S62, S63: Keyswitch, symbol ScottoKeebs:Placeholder_Keyswitch
- added SW1: SW_SPDT, openinput:SW_Micro_Switch, symbol PCM_openinput:SW_SPDT
- added SW2: Switch, symbol ScottoKeebs:Placeholder_Switch
- added SW3: RotaryEncoder_Switch_MP, symbol Device:RotaryEncoder_Switch_MP
- added U1, U4: Nice_Nano_V2, ScottoKeebs_MCU:Nice_Nano_V2, symbol ScottoKeebs:MCU_Nice_Nano_V2
Connections:
- net VCC is gone; now on net +3V3: Display1.3 (VCC), J1.2 (VCC)
- net GND: now also D30.1 (VDD), BT1.2 (-), D100.1 (VDD), D101.1 (VDD), D102.1 (VDD), D103.1 (VDD), D104.1 (VDD), D105.1 (VDD), D106.1 (VDD), D107.1 (VDD), D108.1 (VDD), D109.1 (VDD), D110.1 (VDD), D111.1 (VDD), D112.1 (VDD), D113.1 (VDD), D114.1 (VDD), D115.1 (VDD), D116.1 (VDD), D117.1 (VDD), D118.1 (VDD), D119.1 (VDD), D120.1 (VDD), D121.1 (VDD), D31.1 (VDD), D32.1 (VDD), D33.1 (VDD), D34.1 (VDD), D35.1 (VDD), D36.1 (VDD), D37.1 (VDD), D38.1 (VDD), D39.1 (VDD), D40.1 (VDD), D41.1 (VDD), D42.1 (VDD), D43.1 (VDD), D44.1 (VDD), D45.1 (VDD), D46.1 (VDD), D47.1 (VDD), D48.1 (VDD), D49.1 (VDD), D50.1 (VDD), D51.1 (VDD), D52.1 (VDD), D53.1 (VDD), D54.1 (VDD), D55.1 (VDD), D56.1 (VDD), D57.1 (VDD), D58.1 (VDD), D93.1 (VDD), D94.1 (VDD), D95.1 (VDD), D96.1 (VDD), D97.1 (VDD), D98.1 (VDD), D99.1 (VDD), Display2.4 (GND), J2.1 (GND), U1.23 (GND), U1.3 (GND), U1.4 (GND), U4.23 (GND), U4.3 (GND), U4.4 (GND)
- net at D30.2 (DOUT): now also D31.4 (DIN)
- net +3V3: now reaches D30.3 (VSS)
- net +3V3: now also D100.3 (VSS), D101.3 (VSS), D102.3 (VSS), D103.3 (VSS), D104.3 (VSS), D105.3 (VSS), D106.3 (VSS), D107.3 (VSS), D108.3 (VSS), D109.3 (VSS), D110.3 (VSS), D111.3 (VSS), D112.3 (VSS), D113.3 (VSS), D114.3 (VSS), D115.3 (VSS), D116.3 (VSS), D117.3 (VSS), D118.3 (VSS), D119.3 (VSS), D120.3 (VSS), D121.3 (VSS), D31.3 (VSS), D32.3 (VSS), D33.3 (VSS), D34.3 (VSS), D35.3 (VSS), D36.3 (VSS), D37.3 (VSS), D38.3 (VSS), D39.3 (VSS), D40.3 (VSS), D41.3 (VSS), D42.3 (VSS), D43.3 (VSS), D44.3 (VSS), D45.3 (VSS), D46.3 (VSS), D47.3 (VSS), D48.3 (VSS), D49.3 (VSS), D50.3 (VSS), D51.3 (VSS), D52.3 (VSS), D53.3 (VSS), D54.3 (VSS), D55.3 (VSS), D56.3 (VSS), D57.3 (VSS), D58.3 (VSS), D93.3 (VSS), D94.3 (VSS), D95.3 (VSS), D96.3 (VSS), D97.3 (VSS), D98.3 (VSS), D99.3 (VSS), Display2.3 (VCC), J2.2 (VCC), U1.21 (3.3v), U4.21 (3.3v)
- net COL0 renamed L-COL0
- net L-COL0: now also U4.7 (4)
- net COL1 renamed L-COL1
- net L-COL1: now also U4.8 (5)
- net COL2 renamed L-COL2
- net L-COL2: now also U4.9 (6)
- net COL3 renamed L-COL3
- net L-COL3: now also U4.10 (7)
- net COL4 renamed L-COL4
- net L-COL4: now also U4.11 (8)
- net COL5 renamed L-COL5
- net L-COL5: now also U4.12 (9)
- net CS renamed L-CS
- net L-CS: now also U4.20 (21)
- net RGB renamed L-RGB
- net L-RGB: now also U4.19 (20)
- net ROW0 renamed L-ROW0
- net L-ROW0: now also D59.1 (K), U4.17 (18)
- net ROW1 renamed L-ROW1
- net L-ROW1: now also D60.1 (K), U4.16 (15)
- net ROW2 renamed L-ROW2
- net L-ROW2: now also D61.1 (K), U4.15 (14)
- net ROW3 renamed L-ROW3
- net L-ROW3: now also D62.1 (K), U4.14 (16)
- net ROW4 renamed L-ROW4
- net L-ROW4: now also D63.1 (K), U4.13 (10)
- net SCL renamed L-SCL
- net L-SCL: now also U4.6 (3)
- net SDA renamed L-SDA
- net L-SDA: now also U4.5 (2)
- new net: D33.2 (DOUT), D34.4 (DIN)
- new net: D32.2 (DOUT), D33.4 (DIN)
- new net: D66.2 (A), S37.2
- new net: D43.2 (DOUT), D44.4 (DIN)
- new net: D42.2 (DOUT), D43.4 (DIN)
- new net: D78.2 (A), S49.2
- new net: D35.2 (DOUT), D36.4 (DIN)
- new net: D34.2 (DOUT), D35.4 (DIN)
- new net: D113.4 (DIN), D118.2 (DOUT)
- new net: D117.2 (DOUT), D118.4 (DIN)
- new net: D102.2 (DOUT), D107.4 (DIN)
- new net: D102.4 (DIN), D97.2 (DOUT)
- new net: D44.2 (DOUT), D45.4 (DIN)
- new net: D79.2 (A), S50.2
- new net: D80.2 (A), S51.2
- new net: D105.4 (DIN), D110.2 (DOUT)
- new net: D110.4 (DIN), D115.2 (DOUT)
- new net: D38.2 (DOUT), D39.4 (DIN)
- new net: D37.2 (DOUT), D38.4 (DIN)
- new net: D63.2 (A), S34.2
- new net: D41.2 (DOUT), D42.4 (DIN)
- new net: D40.2 (DOUT), D41.4 (DIN)
- new net: D89.2 (A), S60.2
- new net: D81.2 (A), S52.2
- new net: D74.2 (A), S45.2
- new net: D92.2 (A), S63.2
- new net: D64.2 (A), S35.2
- new net: D94.2 (DOUT), D95.4 (DIN)
- new net: D94.4 (DIN), D98.2 (DOUT)
- new net: D48.2 (DOUT), D49.4 (DIN)
- new net: D47.2 (DOUT), D48.4 (DIN)
- new net: D71.2 (A), S42.2
- new net: D83.2 (A), S54.2
- new net: D88.2 (A), S59.2
- new net: D103.2 (DOUT), D98.4 (DIN)
- new net: D112.2 (DOUT), D117.4 (DIN)
- new net: D73.2 (A), S44.2
- new net: D114.2 (DOUT), D119.4 (DIN)
- new net: D109.2 (DOUT), D114.4 (DIN)
- new net: D31.2 (DOUT), D32.4 (DIN)
- new net: D103.4 (DIN), D108.2 (DOUT)
- new net: D108.4 (DIN), D113.2 (DOUT)
- new net: D85.2 (A), S56.2
- new net: D45.2 (DOUT), D46.4 (DIN)
- new net: SW1.1 (C), U4.24 (B+)
- new net: D62.2 (A), S33.2
- new net: D115.4 (DIN), D120.2 (DOUT)
- new net: D84.2 (A), S55.2
- new net: D59.2 (A), S30.2
- new net: D106.2 (DOUT), D111.4 (DIN)
- new net: D101.2 (DOUT), D106.4 (DIN)
- new net: D67.2 (A), S38.2
- new net: D70.2 (A), S41.2
- new net: D77.2 (A), S48.2
- new net: D36.2 (DOUT), D37.4 (DIN)
- new net: D72.2 (A), S43.2
- new net: D52.2 (DOUT), D53.4 (DIN)
- new net: D51.2 (DOUT), D52.4 (DIN)
- new net: D107.2 (DOUT), D112.4 (DIN)
- new net: D90.2 (A), S61.2
- new net: D61.2 (A), S32.2
- new net: D65.2 (A), S36.2
- new net: D111.2 (DOUT), D116.4 (DIN)
- new net: D68.2 (A), S39.2
- new net: D76.2 (A), S47.2
- new net: D46.2 (DOUT), D47.4 (DIN)
- new net: D104.4 (DIN), D99.2 (DOUT)
- new net: D95.2 (DOUT), D99.4 (DIN)
- new net: D50.2 (DOUT), D51.4 (DIN)
- new net: D49.2 (DOUT), D50.4 (DIN)
- new net: D75.2 (A), S46.2
- new net: D53.2 (DOUT), D54.4 (DIN)
- new net: D56.2 (DOUT), D57.4 (DIN)
- new net: D55.2 (DOUT), D56.4 (DIN)
- new net: D101.4 (DIN), D96.2 (DOUT)
- new net: D86.2 (A), S57.2
- new net: D57.2 (DOUT), D58.4 (DIN)
- new net: D116.2 (DOUT), D121.4 (DIN)
- new net: D119.2 (DOUT), D120.4 (DIN)
- new net: D100.2 (DOUT), D96.4 (DIN)
- new net: D100.4 (DIN), D105.2 (DOUT)
- new net: D104.2 (DOUT), D109.4 (DIN)
- new net: D82.2 (A), S53.2
- new net: D91.2 (A), S62.2
- new net: D69.2 (A), S40.2
- new net: D93.2 (DOUT), D97.4 (DIN)
- new net: D87.2 (A), S58.2
- new net: D60.2 (A), S31.2
- new net: D54.2 (DOUT), D55.4 (DIN)
- new net: D39.2 (DOUT), D40.4 (DIN)
- new net L-BATTERY-POSITIVE: BT1.1 (+), SW1.3 (NC)
- new net L-COL6: S30.1, S31.1, S32.1, S33.1, S34.1
- new net L-ENCODER-A0: SW3.A, U4.1
- new net L-ENCODER-B0: SW3.B, U4.2 (0)
- new net L-RST: U4.22 (RST)
- new net R-COL0: S59.1, S60.1, S61.1, S62.1, U1.18 (19)
- new net R-COL1: S54.1, S55.1, S56.1, S57.1, S63.1, U1.17 (18)
- new net R-COL2: S49.1, S50.1, S51.1, S52.1, S58.1, U1.16 (15)
- new net R-COL3: S44.1, S45.1, S46.1, S47.1, S53.1, U1.15 (14)
- new net R-COL4: S39.1, S40.1, S41.1, S42.1, S48.1, U1.14 (16)
- new net R-COL5: S35.1, S36.1, S37.1, S38.1, S43.1, U1.13 (10)
- new net R-CS: Display2.5 (CS), U1.20 (21)
- new net R-RGB: D93.4 (DIN), U1.19 (20)
- new net R-ROW0: D64.1 (K), D68.1 (K), D73.1 (K), D78.1 (K), D83.1 (K), D88.1 (K), U1.8 (5)
- new net R-ROW1: D65.1 (K), D69.1 (K), D74.1 (K), D79.1 (K), D84.1 (K), D89.1 (K), U1.9 (6)
- new net R-ROW2: D66.1 (K), D70.1 (K), D75.1 (K), D80.1 (K), D85.1 (K), D90.1 (K), U1.10 (7)
- new net R-ROW3: D67.1 (K), D71.1 (K), D76.1 (K), D81.1 (K), D86.1 (K), D91.1 (K), U1.11 (8)
- new net R-ROW4: D72.1 (K), D77.1 (K), D82.1 (K), D87.1 (K), D92.1 (K), U1.12 (9)
- new net R-SCL: Display2.2 (SCK), J2.3 (SCL), U1.6 (3)
- new net R-SDA: Display2.1 (MOSI), J2.4 (SDA), U1.5 (2)
Other:
- note added: "RIGHT SIDE"
- moved on the sheet: D1, D10, D11, D12, D13, D14, D15, D16, D17, D18, D19, D2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

Commit message: minor formatting improvements
Parts:
- added J3: Conn_01x06_Pin, symbol Connector:Conn_01x06_Pin
Other:
- note added: "TPS65 TRACKPAD"
Changed lines of the file:
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@@
 	(generator_version "9.0")
 	(paper "A3")
+	(text "TPS65 TRACKPAD\n"
+		(exclude_from_sim no)
+		(at 290.83 196.088 0)
+		(effects
+			(font
+				(face "KiCad Font")
+				(size 2.54 2.54)
+				(thickness 0.508)
+				(bold yes)
+			)
+		)
+	)
 	(text "Display\n"
 		(exclude_from_sim no)
@@
 					(unit 1)
 				)
+			)
+		)
+	)
+	(symbol
+		(lib_id "Connector:Conn_01x06_Pin")
+		(at 280.67 212.09 0)
+		(unit 1)
+		(exclude_from_sim no)
+		(in_bom yes)
+		(on_board yes)
+		(dnp no)
+		(fields_autoplaced yes)
+		(property "Reference" "J3"
+			(at 281.305 201.93 0)
+			(effects
+				(font
+					(size 1.27 1.27)
+				)
+			)
+		)
+		(property "Value" "Conn_01x06_Pin"
+			(at 281.305 204.47 0)
+			(effects
+				(font
+					(size 1.27 1.27)
+				)
+			)
+		)
+		(property "Footprint" ""
+			(at 280.67 212.09 0)
+			(effects
+				(font
+					(size 1.27 1.27)
+				)
+				(hide yes)
+			)
+		)
+		(property "Datasheet" "~"
+			(at 280.67 212.09 0)
+			(effects
+				(font
+					(size 1.27 1.27)
+				)
+				(hide yes)
+			)
+		)
+		(property "Description" "Generic connector, single row, 01x06, script generated"
+			(at 280.67 212.09 0)
+			(effects
+				(font
+					(size 1.27 1.27)
+				)
+				(hide yes)
+			)
+		)
+		(pin "3"
+		)
+		(pin "4"
+		)
+		(pin "5"
+		)
+		(pin "6"
+		)
+		(pin "2"
+		)
+		(pin "1"
+		)
+		(instances
+			(project ""
+				(path "/a630da1b-27bd-4d59-a0f0-6159ff5296b0"
+					(reference "J3")
+					(unit 1)
+				)
