File: PCB/quartz58.kicad_sch (KiCad schematic)
At the start: 188 parts, among them J1 OLED_128x32, J2 OLED_128x32, SW1 SW_SPDT, SW2 SW_Push_Shielded, SW4 SW_SPDT, SW5 SW_Push_Shielded, T1 TPS65-201A-S, U1 Nice_Nano_V2, U4 Nice_Nano_V2

Commit message: more progress?
Parts:
- BT1, BT2: footprint (none) -> ScottoKeebs_Components:Connector_1x02_JST-PH
- D1, D10, D11, D12, D13, D14, D15, D16, D17, D18, D19, D2, D20, D21, D22, D23, D24, D25, D26, D27, D28, D29, D3, D4, D5, D6, D64, D65, D66, D67, D68, D69, D7, D70, D71, D72, D73, D74, D75, D76, D77, D78, D79, D8, D80, D81, D82, D83, D84, D85, D86, D87, D88, D89, D9, D90, D91, D92: footprint (none) -> ScottoKeebs_Components:Diode_SOD-123
- D100, D101, D102, D103, D104, D105, D106, D107, D108, D109, D110, D111, D112, D113, D114, D115, D116, D117, D118, D119, D120, D121, D30, D31, D32, D33, D34, D35, D36, D37, D38, D39, D40, D41, D42, D43, D44, D45, D46, D47, D48, D49, D50, D51, D52, D53, D54, D55, D56, D57, D58, D93, D94, D95, D96, D97, D98, D99: footprint ScottoKeebs_Components:LED_SK6812MINI -> Keebio-Parts.pretty-master:SK6812-MINI-E
- S1, S10, S11, S12, S13, S14, S15, S16, S17, S18, S19, S2, S20, S21, S22, S23, S24, S25, S26, S27, S28, S29, S3, S35, S36, S37, S38, S39, S4, S40, S41, S42, S43, S44, S45, S46, S47, S48, S49, S5, S50, S51, S52, S53, S54, S55, S56, S57, S58, S59, S6, S60, S61, S62, S63, S7, S8, S9: footprint (none) -> Hotswap_Choc_and_MX:Hotswap_Choc_V1V2
- U1, U4: footprint ScottoKeebs_MCU:Nice_Nano_V2 -> nice-nano-kicad-master:nice_nano

Commit message: coming back
Connections:
- net L-ROW4: no longer E1.6 (SW1)
- net SW1: now reaches U4.25 (1)
- net SW1: now also E1.6 (SW1)
Changed lines of the file:
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@@
+		)
+	)
+	(global_label "SW1"
+		(shape input)
+		(at 45.72 187.96 90)
+		(fields_autoplaced yes)
+		(effects
+			(font
+				(size 1.27 1.27)
+			)
+			(justify left)
+		)
+		(property "Intersheetrefs" "${INTERSHEET_REFS}"
+			(at 45.72 181.1044 90)
+			(effects
+				(font
+					(size 1.27 1.27)
+				)
+				(justify left)
+				(hide yes)
+			)
 		)
 	)
@@
 		)
 	)
+	(global_label "SW1"
+		(shape input)
+		(at 125.73 203.2 180)
+		(fields_autoplaced yes)
+		(effects
+			(font
+				(size 1.27 1.27)
+			)
+			(justify right)
+		)
+		(property "Intersheetrefs" "${INTERSHEET_REFS}"
+			(at 118.8744 203.2 0)
+			(effects
+				(font
+					(size 1.27 1.27)
+				)
+				(justify right)
+				(hide yes)
+			)
+		)
+	)
 	(global_label "R-RGB"
 		(shape input)
@@
 			(effects
 				(font
-					(size 1.27 1.27)
-				)
-				(justify right)
-				(hide yes)
-			)
-		)
-	)
-	(global_label "L-ROW4"
-		(shape input)
-		(at 125.73 203.2 180)
-		(fields_autoplaced yes)
-		(effects
-			(font
-				(size 1.27 1.27)
-			)
-			(justify right)
-		)
-		(property "Intersheetrefs" "${INTERSHEET_REFS}"
-			(at 114.8829 203.2 0)
-			(effects
-				(font

Commit message: pcb and cad updates
Parts:
- removed SW1, SW4: SW_SPDT, openinput:SW_Micro_Switch, symbol PCM_openinput:SW_SPDT
- removed SW2, SW5: SW_Push_Shielded, symbol Switch:SW_Push_Shielded
- added SW2, SW3: SW_Push, ul_EVQ-PUJ02K:SW_EVQPUJ_4P7X3P5_PAN, symbol Switch:SW_Push
- added SW4, SW5: SW_SPDT, SSSS811101:SW_SSSS811101, symbol Switch:SW_SPDT
Connections:
- net GND: now also SW2.1, SW3.1
- net L-BATTERY-POSITIVE: now also SW4.1 (A)
- net L-RST: now also SW3.2
- net R-BATTERY-POSITIVE: now also SW5.1 (A)
- net R-RST: now also SW2.2
- net at U4.24 (B+): now also SW4.2 (B)
- net at U1.24 (B+): now also SW5.2 (B)
Other:
- moved on the sheet: BT1

Commit message: todays progress
Parts:
- added D30, D31, D32, D33: Diode, ScottoKeebs_Components:Diode_SOD-123, symbol ScottoKeebs:Placeholder_Diode
- added J3: Conn_01x10_Socket, Connector_FFC-FPC:Hirose_FH12-10S-0.5SH_1x10-1MP_P0.50mm_Horizontal, symbol Connector:Conn_01x10_Socket
- added J4: Conn_01x10_Pin, Connector_FFC-FPC:Hirose_FH12-10S-0.5SH_1x10-1MP_P0.50mm_Horizontal, symbol Connector:Conn_01x10_Pin
- E1: footprint (none) -> ANO_Encoder:Encoder_TSWB3NCB111LFS
- renumbered D3 to D10, D103 to D100, D108 to D101, D113 to D102, D118 to D103, D95 to D104, D99 to D105, D104 to D106, D109 to D107, D114 to D108, D119 to D109, D9 to D11, D96 to D110, D100 to D111, D105 to D112, D110 to D113, D115 to D114, D120 to D115, D101 to D116, D106 to D117, D111 to D118, D116 to D119, D17 to D12, D121 to D120, D18 to D13, D26 to D14, D4 to D15, D10 to D16, D19 to D17, D20 to D18, D27 to D19, D7 to D2, D5 to D20, D11 to D21, D21 to D22, D22 to D23, D28 to D24, D6 to D25, D12 to D26, D23 to D27, D24 to D28, D13 to D3, D30 to D34, D31 to D35, D32 to D36, D33 to D37, D34 to D38, D35 to D39, D14 to D4, D41 to D40, D40 to D41, D39 to D42, D38 to D43, D37 to D44, D36 to D45, D42 to D46, D43 to D47, D44 to D48, D45 to D49, D2 to D5, D46 to D50, D47 to D51, D53 to D52, D52 to D53, D51 to D54, D50 to D55, D49 to D56, D48 to D57, D54 to D58, D55 to D59, D8 to D6, D56 to D60, D57 to D61, D58 to D62, D64 to D63, D65 to D64, D66 to D65, D67 to D66, D72 to D67, D15 to D7, D77 to D72, D82 to D77, D16 to D8, D87 to D82, D92 to D87, D25 to D9, D93 to D92, D97 to D93, D102 to D94, D107 to D95, D112 to D96, D117 to D97, D94 to D98, D98 to D99, S3 to S10, S9 to S11, S17 to S12, S18 to S13, S26 to S14, S4 to S15, S10 to S16, S19 to S17, S20 to S18, S27 to S19, S7 to S2, S5 to S20, S11 to S21, S21 to S22, S22 to S23, S28 to S24, S6 to S25, S12 to S26, S23 to S27, S24 to S28, S13 to S3, S35 to S30, S36 to S31, S37 to S32, S38 to S33, S43 to S34, S39 to S35, S40 to S36, S41 to S37, S42 to S38, S48 to S39, S14 to S4, S44 to S40, S45 to S41, S46 to S42, S47 to S43, S53 to S44, S49 to S45, S50 to S46, S51 to S47, S52 to S48, S58 to S49, S2 to S5, S54 to S50, S55 to S51, S56 to S52, S57 to S53, S63 to S54, S59 to S55, S60 to S56, S61 to S57, S62 to S58, S8 to S6, S15 to S7, S16 to S8, S25 to S9, SW4 to SW1, SW3 to SW2, SW5 to SW3, SW2 to SW4, U4 to U1, U1 to U2
Connections:
- net GND: now also J3.3 (Pin_3); no longer E1.7 (COMA)
- net L-ENCODER-A0: now also J3.1 (Pin_1); no longer E1.8 (ENCB)
- net L-ENCODER-B0: now also J3.2 (Pin_2); no longer E1.9 (ENCA)
- net L-ROW0: now also D30.1 (K); no longer E1.2 (SW5)
- net L-ROW1: now also D31.1 (K); no longer E1.3 (SW4)
- net L-ROW2: now also D32.1 (K); no longer E1.4 (SW3)
- net L-ROW3: now also D33.1 (K); no longer E1.5 (SW2)
- net SW1: now also J3.4 (Pin_4); no longer E1.6 (SW1)
- net L-COL6: no longer names the net of E1.1 (ENCA)
- net L-COL6: now also J4.1 (Pin_1); no longer U1.18 (19)
- new net: E1.2 (ENCB), J4.2 (Pin_2)
- new net: E1.3 (COMA), J4.3 (Pin_3)
- new net: E1.4 (SW1), J4.4 (Pin_4)
- new net: E1.5 (SW2), J4.5 (Pin_5)
- new net: E1.6 (SW3), J4.6 (Pin_6)
- new net: E1.7 (SW4), J4.7 (Pin_7)
- new net: E1.8 (SW5), J4.8 (Pin_8)
- new net: E1.9 (COMB), J4.9 (Pin_9)
- new net COMB: J3.9 (Pin_9), U1.18 (19)
- new net SW2: D33.2 (A), J3.5 (Pin_5)
- new net SW3: D32.2 (A), J3.6 (Pin_6)
- new net SW4: D31.2 (A), J3.7 (Pin_7)
- new net SW5: D30.2 (A), J3.8 (Pin_8)
Other:
- moved on the sheet: D34, D35, D36, D37, D38, D39, D40, D41, D42, D43, D44, D45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

Commit message: might be cooked chat
Parts:
- U1, U2: footprint nice-nano-kicad-master:nice_nano -> ScottoKeebs_MCU:Nice_Nano_V2_Flipped
Connections:
- net GND: now also SW2.2, SW4.2; no longer SW2.1, SW4.1
- net L-ENCODER-A0: now also U1.2 (0); no longer U1.1
- net L-ENCODER-B0: now also U1.1; no longer U1.2 (0)
- net L-RST: now also SW2.1; no longer SW2.2
- net R-RST: now also SW4.1; no longer SW4.2
Changed lines of the file:
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@@
 		)
 	)
-	(global_label "L-RST"
-		(shape input)
-		(at 92.71 201.93 0)
-		(fields_autoplaced yes)
-		(effects
-			(font
-				(size 1.27 1.27)
-			)
-			(justify left)
-		)
-		(property "Intersheetrefs" "${INTERSHEET_REFS}"
-			(at 99.5052 201.93 0)
-			(effects
-				(font
-					(size 1.27 1.27)
-				)
-				(justify left)
-				(hide yes)
-			)
-		)
-	)
 	(global_label "R-COL1"
 		(shape input)
@@
 		)
 	)
-	(global_label "SW2"
+	(global_label "L-ENCODER-B0"
 		(shape input)
-		(at 93.98 121.92 90)
+		(at 34.29 165.1 180)
 		(fields_autoplaced yes)
 		(effects
@@
 				(size 1.27 1.27)
 			)
-			(justify left)
+			(justify right)
 		)
 		(property "Intersheetrefs" "${INTERSHEET_REFS}"
-			(at 93.98 115.0644 90)
+			(at 15.8834 165.1 0)
 			(effects
 				(font
 					(size 1.27 1.27)
 				)
-				(justify left)
+				(justify right)
 				(hide yes)
 			)
 		)
 	)
-	(global_label "R-CS"
+	(global_label "SW2"
 		(shape input)
-		(at 350.52 240.03 270)
+		(at 93.98 121.92 90)
 		(fields_autoplaced yes)
 		(effects
@@
 				(size 1.27 1.27)
 			)
-			(justify right)
+			(justify left)
 		)
 		(property "Intersheetrefs" "${INTERSHEET_REFS}"
-			(at 350.52 245.4947 90)
+			(at 93.98 115.0644 90)
 			(effects
 				(font
 					(size 1.27 1.27)
 				)
-				(justify right)
+				(justify left)
 				(hide yes)
 			)
 		)
 	)
-	(global_label "L-ENCODER-B0"
+	(global_label "R-CS"
 		(shape input)
-		(at 34.29 167.64 180)
+		(at 350.52 240.03 270)
 		(fields_autoplaced yes)
 		(effects
@@
 		)
 		(property "Intersheetrefs" "${INTERSHEET_REFS}"
-			(at 15.8834 167.64 0)
+			(at 350.52 245.4947 90)
 			(effects
 				(font
@@
 		)
 	)
+	(global_label "L-ENCODER-A0"
+		(shape input)
+		(at 34.29 167.64 180)
+		(fields_autoplaced yes)
+		(effects
+			(font
+				(size 1.27 1.27)
+			)
+			(justify right)
+		)
+		(property "Intersheetrefs" "${INTERSHEET_REFS}"
+			(at 16.0648 167.64 0)
+			(effects
+				(font
+					(size 1.27 1.27)
+				)
+				(justify right)
+				(hide yes)
+			)
+		)
+	)
 	(global_label "L-COL6"
 		(shape input)
@@
 		)
 	)
-	(global_label "L-ENCODER-A0"
+	(global_label "R-RST"
 		(shape input)
-		(at 34.29 165.1 180)
+		(at 373.38 210.82 180)
 		(fields_autoplaced yes)
 		(effects
@@
 		)
 		(property "Intersheetrefs" "${INTERSHEET_REFS}"
-			(at 16.0648 165.1 0)
+			(at 364.1053 210.82 0)
 			(effects
 				(font
@@
 		)
 	)
+	(global_label "L-RST"
+		(shape input)
+		(at 82.55 201.93 180)
+		(fields_autoplaced yes)
+		(effects
+			(font
+				(size 1.27 1.27)
+			)
+			(justify right)
+		)
+		(property "Intersheetrefs" "${INTERSHEET_REFS}"
+			(at 73.5172 201.93 0)
+			(effects
+				(font
+					(size 1.27 1.27)
+				)
+				(justify right)
+				(hide yes)
+			)
+		)
+	)
 	(global_label "R-COL3"
 		(shape input)
@@
 		)
 	)
-	(global_label "R-RST"
-		(shape input)
-		(at 383.54 210.82 0)
-		(fields_autoplaced yes)
-		(effects
-			(font
-				(size 1.27 1.27)
-			)
-			(justify left)
-		)
-		(property "Intersheetrefs" "${INTERSHEET_REFS}"
-			(at 390.3352 210.82 0)
-			(effects
-				(font
-					(size 1.27 1.27)
-				)
-				(justify left)
-				(hide yes)
-			)
-		)
-	)
 	(global_label "R-RGB"
 		(shape input)
@@
 			)
 		)
-		(property "Footprint" "nice-nano-kicad-master:nice_nano"
+		(property "Footprint" "ScottoKeebs_MCU:Nice_Nano_V2_Flipped"
 			(at 49.53 201.93 0)
 			(effects
@@
 	(symbol
 		(lib_id "power:GND")
-		(at 82.55 201.93 270)
+		(at 92.71 201.93 90)
 		(unit 1)
 		(exclude_from_sim no)
@@
 		(fields_autoplaced yes)
 		(property "Reference" "#PWR07"
-			(at 76.2 201.93 0)
+			(at 99.06 201.93 0)
 			(effects
 				(font
@@
 		)
 		(property "Value" "GND"
-			(at 78.74 201.9299 90)
+			(at 96.52 201.9299 90)
 			(effects
 				(font
@@
 		)
 		(property "Footprint" ""
-			(at 82.55 201.93 0)
+			(at 92.71 201.93 0)
 			(effects
 				(font
@@
 		)
 		(property "Datasheet" ""
-			(at 82.55 201.93 0)
+			(at 92.71 201.93 0)
 			(effects
 				(font
@@
 		)
 		(property "Description" "Power symbol creates a global label with name \"GND\" , ground"
-			(at 82.55 201.93 0)
+			(at 92.71 201.93 0)
 			(effects
 				(font
@@
 	)
 	(symbol
+		(lib_id "power:GND")
+		(at 383.54 210.82 90)
+		(unit 1)
+		(exclude_from_sim no)
+		(in_bom yes)
+		(on_board yes)
+		(dnp no)
+		(fields_autoplaced yes)
+		(property "Reference" "#PWR024"
+			(at 389.89 210.82 0)
+			(effects
+				(font
+					(size 1.27 1.27)
+				)
+				(hide yes)
+			)
+		)
+		(property "Value" "GND"
+			(at 387.35 210.8199 90)
+			(effects
+				(font
+					(size 1.27 1.27)
+				)
+				(justify right)
+			)
+		)
+		(property "Footprint" ""
+			(at 383.54 210.82 0)
+			(effects
+				(font
+					(size 1.27 1.27)
+				)
+				(hide yes)
+			)
+		)
+		(property "Datasheet" ""
+			(at 383.54 210.82 0)
+			(effects
+				(font
+					(size 1.27 1.27)
+				)
+				(hide yes)
+			)
+		)
+		(property "Description" "Power symbol creates a global label with name \"GND\" , ground"
+			(at 383.54 210.82 0)
+			(effects
+				(font
+					(size 1.27 1.27)
+				)
+				(hide yes)
+			)
+		)
+		(pin "1"
+		)
+		(instances
+			(project "quartz58"
+				(path "/a630da1b-27bd-4d59-a0f0-6159ff5296b0"
+					(reference "#PWR024")
+					(unit 1)
+				)
+			)
+		)
+	)
+	(symbol
 		(lib_id "ScottoKeebs:OLED_128x32")
 		(at 35.56 231.14 90)
@@
 	)
 	(symbol
-		(lib_id "power:GND")
-		(at 373.38 210.82 270)
-		(unit 1)
-		(exclude_from_sim no)
-		(in_bom yes)
-		(on_board yes)
-		(dnp no)
-		(fields_autoplaced yes)
-		(property "Reference" "#PWR022"
-			(at 367.03 210.82 0)
-			(effects
-				(font
-					(size 1.27 1.27)
-				)
-				(hide yes)
-			)
-		)
-		(property "Value" "GND"
-			(at 369.57 210.8199 90)
-			(effects
-				(font
-					(size 1.27 1.27)
-				)
-				(justify right)
-			)
-		)
-		(property "Footprint" ""
-			(at 373.38 210.82 0)
-			(effects
-				(font
-					(size 1.27 1.27)
-				)
-				(hide yes)
-			)
-		)
-		(property "Datasheet" ""
-			(at 373.38 210.82 0)
-			(effects
-				(font
-					(size 1.27 1.27)
-				)
-				(hide yes)
-			)
-		)
-		(property "Description" "Power symbol creates a global label with name \"GND\" , ground"
-			(at 373.38 210.82 0)
-			(effects
-				(font
-					(size 1.27 1.27)
-				)
-				(hide yes)
-			)
-		)
-		(pin "1"
-		)
-		(instances
-			(project "quartz58"
-				(path "/a630da1b-27bd-4d59-a0f0-6159ff5296b0"
-					(reference "#PWR022")
-					(unit 1)
-				)
-			)
-		)
-	)
-	(symbol
 		(lib_id "ScottoKeebs:LED_SK6812MINI")
 		(at 332.74 146.05 0)
@@
 			)
 		)
-		(property "Footprint" "nice-nano-kicad-master:nice_nano"
+		(property "Footprint" "ScottoKeebs_MCU:Nice_Nano_V2_Flipped"
 			(at 344.17 205.74 0)
 			(effects

Commit message: todays progress
Connections:
- net at J4.1 (Pin_1): no longer E1.1 (ENCA)
- net at J4.10 (Pin_10): now also E1.1 (ENCA)
- net at J4.2 (Pin_2): now also E1.9 (COMB); no longer E1.2 (ENCB)
- net at J4.3 (Pin_3): now also E1.8 (SW5); no longer E1.3 (COMA)
- net at J4.4 (Pin_4): now also E1.7 (SW4); no longer E1.4 (SW1)
- net at J4.5 (Pin_5): now also E1.6 (SW3); no longer E1.5 (SW2)
- net at J4.6 (Pin_6): now also E1.5 (SW2); no longer E1.6 (SW3)
- net at J4.7 (Pin_7): now also E1.4 (SW1); no longer E1.7 (SW4)
- net at J4.8 (Pin_8): now also E1.3 (COMA); no longer E1.8 (SW5)
- net at J4.9 (Pin_9): now also E1.2 (ENCB); no longer E1.9 (COMB)
Other:
- moved on the sheet: E1, J4
Changed lines of the file:
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@@
 	(symbol
 		(lib_id "Connector:Conn_01x10_Pin")
-		(at 160.02 203.2 0)
+		(at 160.02 200.66 0)
+		(mirror x)
 		(unit 1)
 		(exclude_from_sim no)
@@
 		(on_board yes)
 		(dnp no)
-		(fields_autoplaced yes)
 		(property "Reference" "J4"
-			(at 160.655 187.96 0)
-			(effects
-				(font
-					(size 1.27 1.27)
-				)
+			(at 158.75 198.1199 0)
+			(effects
+				(font
+					(size 1.27 1.27)
+				)
+				(justify right)
 			)
 		)
 		(property "Value" "Conn_01x10_Pin"
-			(at 160.655 190.5 0)
-			(effects
-				(font
-					(size 1.27 1.27)
-				)
+			(at 158.75 200.6599 0)
+			(effects
+				(font
+					(size 1.27 1.27)
+				)
+				(justify right)
 			)
 		)
 		(property "Footprint" "Connector_FFC-FPC:Hirose_FH12-10S-0.5SH_1x10-1MP_P0.50mm_Horizontal"
-			(at 160.02 203.2 0)
+			(at 160.02 200.66 0)
 			(effects
 				(font
@@
 		)
 		(property "Datasheet" "~"
-			(at 160.02 203.2 0)
+			(at 160.02 200.66 0)
 			(effects
 				(font
@@
 		)
 		(property "Description" "Generic connector, single row, 01x10, script generated"
-			(at 160.02 203.2 0)
+			(at 160.02 200.66 0)
 			(effects
 				(font
@@
 		)
 		(instances
-			(project ""
+			(project "quartz58"
 				(path "/a630da1b-27bd-4d59-a0f0-6159ff5296b0"
 					(reference "J4")
@@
 	(symbol
 		(lib_id "Encoder_TSWB3NCB111LFS:TSWB3NCB111LFS")
-		(at 170.18 203.2 0)
+		(at 170.18 198.12 0)
 		(unit 1)
 		(exclude_from_sim no)
@@
 		(fields_autoplaced yes)
 		(property "Reference" "E1"
-			(at 176.53 201.9299 0)
+			(at 176.53 196.8499 0)
 			(effects
 				(font
@@
 		)
 		(property "Value" "TSWB3NCB111LFS"
-			(at 176.53 204.4699 0)
+			(at 176.53 199.3899 0)
 			(effects
 				(font
@@
 		)
 		(property "Footprint" "ANO_Encoder:Encoder_TSWB3NCB111LFS"
-			(at 170.18 203.2 0)
+			(at 170.18 198.12 0)
 			(effects
 				(font
@@
 		)
 		(property "Datasheet" ""
-			(at 170.18 203.2 0)
+			(at 170.18 198.12 0)
 			(effects
 				(font
@@
 		)
 		(property "Description" ""
-			(at 170.18 203.2 0)
-			(effects
-				(font
+			(at 170.18 198.12 0)
+			(effects
+				(font

Commit message: more progress
Connections:
- net L-CS: now also U1.2 (0); no longer U1.20 (21)
- net L-ENCODER-A0: now also U1.19 (20); no longer U1.2 (0)
- net L-ENCODER-B0: now also U1.20 (21); no longer U1.1
- net L-RGB: now also U1.1; no longer U1.19 (20)
- net R-COL0: now also S30.1, S31.1, S32.1, S33.1, S34.1, U2.13 (10); no longer S55.1, S56.1, S57.1, S58.1, U2.18 (19)
- net R-COL1: now also S35.1, S36.1, S37.1, S38.1, S39.1, U2.14 (16); no longer S50.1, S51.1, S52.1, S53.1, S54.1, U2.17 (18)
- net R-COL2: now also S40.1, S41.1, S42.1, S43.1, S44.1, U2.15 (14); no longer S45.1, S46.1, S47.1, S48.1, S49.1, U2.16 (15)
- net R-COL3: now also S45.1, S46.1, S47.1, S48.1, S49.1, U2.16 (15); no longer S40.1, S41.1, S42.1, S43.1, S44.1, U2.15 (14)
- net R-COL4: now also S50.1, S51.1, S52.1, S53.1, S54.1, U2.17 (18); no longer S35.1, S36.1, S37.1, S38.1, S39.1, U2.14 (16)
- net R-COL5: now also S55.1, S56.1, S57.1, S58.1, U2.18 (19); no longer S30.1, S31.1, S32.1, S33.1, S34.1, U2.13 (10)
- net R-CS: now also U2.2 (0); no longer U2.20 (21)
- net R-RDY: now also U2.19 (20); no longer U2.2 (0)
- net R-RGB: now also U2.1; no longer U2.19 (20)

Commit message: left side ready for review
Connections:
- net COMB: now also U1.7 (4); no longer U1.18 (19)
- net L-COL0: now also U1.17 (18); no longer U1.7 (4)
- net L-COL1: now also U1.16 (15); no longer U1.8 (5)
- net L-COL2: now also U1.15 (14); no longer U1.9 (6)
- net L-COL3: now also U1.14 (16); no longer U1.10 (7)
- net L-COL4: now also U1.13 (10); no longer U1.11 (8)
- net L-COL5: now also U1.18 (19); no longer U1.12 (9)
- net L-ROW0: now also U1.8 (5); no longer U1.17 (18)
- net L-ROW1: now also U1.9 (6); no longer U1.16 (15)
- net L-ROW2: now also U1.10 (7); no longer U1.15 (14)
- net L-ROW3: now also U1.11 (8); no longer U1.14 (16)
- net L-ROW4: now also U1.12 (9); no longer U1.13 (10)
- net +3V8: now reaches SW3.2 (B), U2.24 (B+)
