File: PCB/quartz58.kicad_pcb (KiCad board)
At the start: 2 copper layers, 277 x 110.9 mm, 177 parts, among them J1 OLED_128x32, J2 OLED_128x32, U1 Nice_Nano_V2, U4 Nice_Nano_V2

Commit message: coming back
Parts:
- moved BT1 64.8 mm to (199.9, 111.1)
- moved Display1 64.8 mm to (199.9, 125.1)
- moved J1 64.8 mm to (193.8, 145.4)
- moved U4 64.8 mm to (199.9, 124.9)
Other:
- outline, holes or cut-outs redrawn
Changed lines of the file:
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@@
 		(0 "F.Cu" signal)
 		(2 "B.Cu" signal)
-		(9 "F.Adhes" user)
-		(11 "B.Adhes" user)
+		(9 "F.Adhes" user "F.Adhesive")
+		(11 "B.Adhes" user "B.Adhesive")
 		(13 "F.Paste" user)
 		(15 "B.Paste" user)
-		(5 "F.SilkS" user)
-		(7 "B.SilkS" user)
+		(5 "F.SilkS" user "F.Silkscreen")
+		(7 "B.SilkS" user "B.Silkscreen")
 		(1 "F.Mask" user)
 		(3 "B.Mask" user)
-		(17 "Dwgs.User" user)
-		(19 "Cmts.User" user)
-		(21 "Eco1.User" user)
-		(23 "Eco2.User" user)
+		(17 "Dwgs.User" user "User.Drawings")
+		(19 "Cmts.User" user "User.Comments")
+		(21 "Eco1.User" user "User.Eco1")
+		(23 "Eco2.User" user "User.Eco2")
 		(25 "Edge.Cuts" user)
 		(27 "Margin" user)
-		(31 "F.CrtYd" user)
-		(29 "B.CrtYd" user)
+		(31 "F.CrtYd" user "F.Courtyard")
+		(29 "B.CrtYd" user "B.Courtyard")
 		(35 "F.Fab" user)
 		(33 "B.Fab" user)
@@
 		(allow_soldermask_bridges_in_footprints no)
 		(tenting front back)
-		(grid_origin 75.009438 111.918844)
+		(grid_origin 189.309446 106.918852)
 		(pcbplotparams
 			(layerselection 0x00000000_00000000_55555555_5755f5ff)
@@
 	(footprint "nice_view:nice_view"
 		(layer "F.Cu")
-		(at 200.849021 60.384462)
+		(at 199.909029 125.14447)
 		(property "Reference" "Display1"
 			(at 0 1.27 0)
@@
 	(footprint "ScottoKeebs_Components:OLED_128x32"
 		(layer "F.Cu")
-		(at 194.769021 80.594462 90)
+		(at 193.829029 145.35447 90)
 		(property "Reference" "J1"
 			(at 7.75 10 90)
@@
 	(footprint "ScottoKeebs_Components:Connector_1x02_JST-PH"
 		(layer "B.Cu")
-		(at 200.799021 46.364462 180)
+		(at 199.859029 111.12447 180)
 		(property "Reference" "BT1"
 			(at 0 6.93 0)
@@
 	(footprint "nice-nano-kicad-master:nice_nano"
 		(layer "B.Cu")
-		(at 200.869438 60.128844 -90)
+		(at 199.929446 124.888852 -90)
 		(property "Reference" "U4"
 			(at 0 -1.625 90)
@@
 	)
 	(gr_line
-		(start 210.931468 101.918844)
-		(end 210.859446 153.543852)
+		(start 210.831059 101.918852)
+		(end 210.759037 153.54386)
 		(stroke
 			(width 0.15)

Commit message: pcb and cad updates
Parts:
- removed D1, D10, D11, D12, D14, D15, D16, D17, D18, D19, D2, D20, D22, D23, D24, D25, D26, D3, D4, D5, D6, D64, D65, D66, D67, D68, D69, D7, D70, D71, D72, D73, D74, D75, D76, D77, D78, D79, D8, D80, D81, D82, D83, D84, D85, D86, D87, D88, D89, D9, D90, D91, D92: Diode, ScottoKeebs_Components:Diode_SOD-123
- removed D100, D101, D102, D103, D104, D105, D106, D107, D108, D109, D110, D111, D112, D113, D114, D115, D116, D117, D118, D119, D120, D121, D30, D31, D32, D33, D34, D35, D36, D37, D38, D39, D40, D41, D42, D43, D44, D45, D46, D47, D48, D49, D50, D51, D52, D53, D54, D55, D56, D57, D58, D93, D94, D95, D96, D97, D98, D99: LED_SK6812MINI, Keebio-Parts.pretty-master:SK6812-MINI-E
- removed S59, S60, S61, S62, S63: Keyswitch, Hotswap_Choc_and_MX:Hotswap_Choc_V1V2
- added LED1: , Keebio-Parts.pretty-master:SK6812-MINI-E, F.Cu at (56.0, 156.6)
- added LED10: , Keebio-Parts.pretty-master:SK6812-MINI-E, F.Cu at (94.1, 129.6)
- added LED11: , Keebio-Parts.pretty-master:SK6812-MINI-E, F.Cu at (94.1, 110.5)
- added LED12: , Keebio-Parts.pretty-master:SK6812-MINI-E, F.Cu at (94.1, 91.5)
- added LED13: , Keebio-Parts.pretty-master:SK6812-MINI-E, F.Cu at (113.1, 146.6)
- added LED14: , Keebio-Parts.pretty-master:SK6812-MINI-E, F.Cu at (113.1, 127.6)
- added LED15: , Keebio-Parts.pretty-master:SK6812-MINI-E, F.Cu at (113.1, 108.5)
- added LED16: , Keebio-Parts.pretty-master:SK6812-MINI-E, F.Cu at (113.1, 89.5)
- added LED17: , Keebio-Parts.pretty-master:SK6812-MINI-E, F.Cu at (132.2, 148.6)
- added LED18: , Keebio-Parts.pretty-master:SK6812-MINI-E, F.Cu at (132.2, 129.6)
- added LED19: , Keebio-Parts.pretty-master:SK6812-MINI-E, F.Cu at (132.2, 110.5)
- added LED2: , Keebio-Parts.pretty-master:SK6812-MINI-E, F.Cu at (56.0, 137.6)
- added LED20: , Keebio-Parts.pretty-master:SK6812-MINI-E, F.Cu at (132.2, 91.5)
- added LED21: , Keebio-Parts.pretty-master:SK6812-MINI-E, F.Cu at (151.2, 151.6)
- added LED22: , Keebio-Parts.pretty-master:SK6812-MINI-E, F.Cu at (151.2, 132.6)
- added LED23: , Keebio-Parts.pretty-master:SK6812-MINI-E, F.Cu at (151.2, 113.5)
- added LED24: , Keebio-Parts.pretty-master:SK6812-MINI-E, F.Cu at (151.2, 94.5)
- added LED25: , Keebio-Parts.pretty-master:SK6812-MINI-E, F.Cu at (170.3, 142.1)
- added LED26: , Keebio-Parts.pretty-master:SK6812-MINI-E, F.Cu at (103.6, 167.7)
- added LED27: , Keebio-Parts.pretty-master:SK6812-MINI-E, F.Cu at (122.6, 167.7)
- added LED28: , Keebio-Parts.pretty-master:SK6812-MINI-E, F.Cu at (141.7, 170.7)
- added LED29: , Keebio-Parts.pretty-master:SK6812-MINI-E, F.Cu at (170.7, 168.7)
- added LED3: , Keebio-Parts.pretty-master:SK6812-MINI-E, F.Cu at (56.0, 118.5)
- added LED30: , Keebio-Parts.pretty-master:SK6812-MINI-E, F.Cu at (370.3, 156.6)
- added LED31: , Keebio-Parts.pretty-master:SK6812-MINI-E, F.Cu at (370.3, 137.6)
- added LED32: , Keebio-Parts.pretty-master:SK6812-MINI-E, F.Cu at (370.3, 118.5)
- added LED33: , Keebio-Parts.pretty-master:SK6812-MINI-E, F.Cu at (370.3, 99.5)
- added LED34: , Keebio-Parts.pretty-master:SK6812-MINI-E, F.Cu at (351.2, 153.6)
- added LED35: , Keebio-Parts.pretty-master:SK6812-MINI-E, F.Cu at (351.2, 134.6)
- added LED36: , Keebio-Parts.pretty-master:SK6812-MINI-E, F.Cu at (351.2, 115.5)
- added LED37: , Keebio-Parts.pretty-master:SK6812-MINI-E, F.Cu at (351.2, 96.5)
- added LED38: , Keebio-Parts.pretty-master:SK6812-MINI-E, F.Cu at (332.2, 148.6)
- added LED39: , Keebio-Parts.pretty-master:SK6812-MINI-E, F.Cu at (332.2, 129.6)
- added LED4: , Keebio-Parts.pretty-master:SK6812-MINI-E, F.Cu at (56.0, 99.5)
- added LED40: , Keebio-Parts.pretty-master:SK6812-MINI-E, F.Cu at (332.2, 110.5)
- added LED41: , Keebio-Parts.pretty-master:SK6812-MINI-E, F.Cu at (332.2, 91.5)
- added LED42: , Keebio-Parts.pretty-master:SK6812-MINI-E, F.Cu at (313.1, 146.6)
- added LED43: , Keebio-Parts.pretty-master:SK6812-MINI-E, F.Cu at (313.1, 127.6)
- added LED44: , Keebio-Parts.pretty-master:SK6812-MINI-E, F.Cu at (313.1, 108.5)
- added LED45: , Keebio-Parts.pretty-master:SK6812-MINI-E, F.Cu at (313.1, 89.5)
- added LED46: , Keebio-Parts.pretty-master:SK6812-MINI-E, F.Cu at (294.1, 148.6)
- added LED47: , Keebio-Parts.pretty-master:SK6812-MINI-E, F.Cu at (294.1, 129.6)
- added LED48: , Keebio-Parts.pretty-master:SK6812-MINI-E, F.Cu at (294.1, 110.5)
- added LED49: , Keebio-Parts.pretty-master:SK6812-MINI-E, F.Cu at (294.1, 91.5)
- added LED5: , Keebio-Parts.pretty-master:SK6812-MINI-E, F.Cu at (75.0, 153.6)
- added LED50: , Keebio-Parts.pretty-master:SK6812-MINI-E, F.Cu at (275.0, 151.6)
- added LED51: , Keebio-Parts.pretty-master:SK6812-MINI-E, F.Cu at (275.0, 132.6)
- added LED52: , Keebio-Parts.pretty-master:SK6812-MINI-E, F.Cu at (275.0, 113.5)
- added LED53: , Keebio-Parts.pretty-master:SK6812-MINI-E, F.Cu at (275.0, 94.5)
- added LED54: , Keebio-Parts.pretty-master:SK6812-MINI-E, F.Cu at (256.0, 142.1)
- added LED55: , Keebio-Parts.pretty-master:SK6812-MINI-E, F.Cu at (322.7, 167.7)
- added LED56: , Keebio-Parts.pretty-master:SK6812-MINI-E, F.Cu at (303.6, 167.7)
- added LED57: , Keebio-Parts.pretty-master:SK6812-MINI-E, F.Cu at (284.6, 170.7)
- added LED58: , Keebio-Parts.pretty-master:SK6812-MINI-E, F.Cu at (255.6, 168.7)
- added LED6: , Keebio-Parts.pretty-master:SK6812-MINI-E, F.Cu at (75.0, 134.6)
- added LED7: , Keebio-Parts.pretty-master:SK6812-MINI-E, F.Cu at (75.0, 115.5)
- added LED8: , Keebio-Parts.pretty-master:SK6812-MINI-E, F.Cu at (75.0, 96.5)
- added LED9: , Keebio-Parts.pretty-master:SK6812-MINI-E, F.Cu at (94.1, 148.6)
- added S30: , comboswitch:Hotswap_Choc_V1V2, F.Cu at (370.3, 152.1)
- added S31: , comboswitch:Hotswap_Choc_V1V2, F.Cu at (370.3, 133.1)
- added S32: , comboswitch:Hotswap_Choc_V1V2, F.Cu at (370.3, 114.0)
- added S33: , comboswitch:Hotswap_Choc_V1V2, F.Cu at (370.3, 95.0)
- added S34: , comboswitch:Hotswap_Choc_V1V2, F.Cu at (351.2, 149.1)
- S1, S10, S11, S12, S13, S14, S15, S16, S17, S18, S19, S2, S20, S21, S22, S23, S24, S25, S26, S29, S3, S35, S36, S37, S38, S39, S4, S40, S41, S42, S43, S44, S45, S46, S47, S49, S5, S50, S51, S52, S54, S55, S56, S57, S58, S6, S7, S8, S9: value Keyswitch -> (none); footprint Hotswap_Choc_and_MX:Hotswap_Choc_V1V2 -> comboswitch:Hotswap_Choc_V1V2
- S27, S28, S48, S53: footprint Hotswap_Choc_and_MX:Hotswap_Choc_V1V2 -> comboswitch:Hotswap_Choc_V1V2
- moved S37 122.0 mm to (351.2, 92.0)
- moved S36 107.6 mm to (351.2, 111.0)
- moved S48 107.5 mm to (294.1, 106.0), turned to 0 degrees
- moved S6 105.7 mm to (75.0, 130.1)
- moved S35 105.6 mm to (351.2, 130.1)
- moved S53 104.4 mm to (275.0, 90.0)
- moved S12 98.5 mm to (94.1, 87.0)
- moved S43 95.0 mm to (313.1, 123.1)
- moved S5 92.9 mm to (75.0, 149.1)
- moved S41 92.8 mm to (332.2, 87.0)
- moved S16 91.1 mm to (113.1, 85.0)
- moved S38 90.6 mm to (332.2, 144.1)
- moved S24 88.4 mm to (151.2, 90.0)
- moved S4 87.3 mm to (56.0, 95.0)
- moved S20 82.2 mm to (132.2, 87.0)
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Connections:
- net Net-(D13-A) renamed middle_bottom
- net Net-(D21-A) renamed inner_bottom
- S1 pad 1: L-COL0 -> (no net)
- S1 pad 2: Net-(D1-A) -> outer_bottom
- S10 pad 1: L-COL3 -> (no net)
- S10 pad 2: Net-(D10-A) -> ring_home
- S11 pad 1: L-COL4 -> (no net)
- S11 pad 2: Net-(D11-A) -> ring_top
- S12 pad 1: L-COL5 -> (no net)
- S12 pad 2: Net-(D12-A) -> ring_stretch
- S13 pad 1: L-COL0 -> (no net)
- S14 pad 1: L-COL0 -> (no net)
- S14 pad 2: Net-(D14-A) -> middle_home
- S15 pad 1: L-COL1 -> (no net)
- S15 pad 2: Net-(D15-A) -> middle_top
- S16 pad 1: L-COL1 -> (no net)
- S16 pad 2: Net-(D16-A) -> middle_stretch
- S17 pad 1: L-COL2 -> (no net)
- S17 pad 2: Net-(D17-A) -> index_bottom
- S18 pad 1: L-COL2 -> (no net)
- S18 pad 2: Net-(D18-A) -> index_home
- S19 pad 1: L-COL3 -> (no net)
- S19 pad 2: Net-(D19-A) -> index_top
- S2 pad 1: L-COL1 -> (no net)
- S2 pad 2: Net-(D2-A) -> outer_home
- S20 pad 1: L-COL3 -> (no net)
- S20 pad 2: Net-(D20-A) -> index_stretch
- S21 pad 1: L-COL4 -> (no net)
- S22 pad 1: L-COL4 -> (no net)
- S22 pad 2: Net-(D22-A) -> inner_home
- S23 pad 1: L-COL5 -> (no net)
- S23 pad 2: Net-(D23-A) -> inner_top
- S24 pad 1: L-COL5 -> (no net)
- S24 pad 2: Net-(D24-A) -> inner_stretch
- S25 pad 1: L-COL1 -> (no net)
- S25 pad 2: Net-(D25-A) -> reach_reach
- S26 pad 1: L-COL2 -> (no net)
- S26 pad 2: Net-(D26-A) -> tucky1_stretch
- S27 pad 2: tucky3_stretch -> tucky2_stretch
- S28 pad 2: reachy_stretch -> tucky3_stretch
- S29 pad 1: L-COL5 -> (no net)
- S29 pad 2: Net-(D29-A) -> reachy_stretch
- S3 pad 1: L-COL2 -> (no net)
- S3 pad 2: Net-(D3-A) -> outer_top
- S35 pad 1: R-COL5 -> (no net)
- S35 pad 2: Net-(D64-A) -> mirror_pinky_home
- S36 pad 1: R-COL5 -> (no net)
- S36 pad 2: Net-(D65-A) -> mirror_pinky_top
- S37 pad 1: R-COL5 -> (no net)
- S37 pad 2: Net-(D66-A) -> mirror_pinky_stretch
- S38 pad 1: R-COL5 -> (no net)
- S38 pad 2: Net-(D67-A) -> mirror_ring_bottom
- S39 pad 1: R-COL4 -> (no net)
- S39 pad 2: Net-(D68-A) -> mirror_ring_home
- S4 pad 1: L-COL3 -> (no net)
- S4 pad 2: Net-(D4-A) -> outer_stretch
- S40 pad 1: R-COL4 -> (no net)
- S40 pad 2: Net-(D69-A) -> mirror_ring_top
- S41 pad 1: R-COL4 -> (no net)
- S41 pad 2: Net-(D70-A) -> mirror_ring_stretch
- S42 pad 1: R-COL4 -> (no net)
- S42 pad 2: Net-(D71-A) -> mirror_middle_bottom
- S43 pad 1: R-COL5 -> (no net)
- S43 pad 2: Net-(D72-A) -> mirror_middle_home
- S44 pad 1: R-COL3 -> (no net)
- S44 pad 2: Net-(D73-A) -> mirror_middle_top
- S45 pad 1: R-COL3 -> (no net)
- S45 pad 2: Net-(D74-A) -> mirror_middle_stretch
- S46 pad 1: R-COL3 -> (no net)
- S46 pad 2: Net-(D75-A) -> mirror_index_bottom
- S47 pad 1: R-COL3 -> (no net)
- S47 pad 2: Net-(D76-A) -> mirror_index_home
- S48 pad 2: mirror_reachy_stretch -> mirror_index_top
- S49 pad 1: R-COL2 -> (no net)
- S49 pad 2: Net-(D78-A) -> mirror_index_stretch
- S5 pad 1: L-COL4 -> (no net)
- S5 pad 2: Net-(D5-A) -> pinky_bottom
- S50 pad 1: R-COL2 -> (no net)
- S50 pad 2: Net-(D79-A) -> mirror_inner_bottom
- S51 pad 1: R-COL2 -> (no net)
- S51 pad 2: Net-(D80-A) -> mirror_inner_home
- S52 pad 1: R-COL2 -> (no net)
- S52 pad 2: Net-(D81-A) -> mirror_inner_top
- S53 pad 2: mirror_tucky3_stretch -> mirror_inner_stretch
- S54 pad 1: R-COL1 -> (no net)
- S54 pad 2: Net-(D83-A) -> mirror_reach_reach
- S55 pad 1: R-COL1 -> (no net)
- S55 pad 2: Net-(D84-A) -> mirror_tucky1_stretch
- S56 pad 1: R-COL1 -> (no net)
- S56 pad 2: Net-(D85-A) -> mirror_tucky2_stretch
- S57 pad 1: R-COL1 -> (no net)
- S57 pad 2: Net-(D86-A) -> mirror_tucky3_stretch
- S58 pad 1: R-COL2 -> (no net)
- S58 pad 2: Net-(D87-A) -> mirror_reachy_stretch
- S6 pad 1: L-COL5 -> (no net)
- S6 pad 2: Net-(D6-A) -> pinky_home
- S7 pad 1: L-COL0 -> (no net)
- S7 pad 2: Net-(D7-A) -> pinky_top
- S8 pad 1: L-COL1 -> (no net)
- S8 pad 2: Net-(D8-A) -> pinky_stretch
- S9 pad 1: L-COL2 -> (no net)
- S9 pad 2: Net-(D9-A) -> ring_bottom
Routing:
- net Net-(D1-A): track 3.02 -> 0.00 mm
Other:
- board size 277 x 110.9 mm -> 334.4 x 109.5 mm

Commit message: todays progress
Parts:
- removed LED1, LED10, LED11, LED12, LED13, LED14, LED15, LED16, LED17, LED18, LED19, LED2, LED20, LED21, LED22, LED23, LED24, LED25, LED26, LED27, LED28, LED29, LED3, LED30, LED31, LED32, LED33, LED34, LED35, LED36, LED37, LED38, LED39, LED4, LED40, LED41, LED42, LED43, LED44, LED45, LED46, LED47, LED48, LED49, LED5, LED50, LED51, LED52, LED53, LED54, LED55, LED56, LED57, LED58, LED6, LED7, LED8, LED9: , Keebio-Parts.pretty-master:SK6812-MINI-E
- added D1: Diode, ScottoKeebs_Components:Diode_SOD-123, B.Cu at (63.1, 102.7)
- added D10: Diode, ScottoKeebs_Components:Diode_SOD-123, B.Cu at (101.2, 94.3)
- added D100: LED_SK6812MINI, Keebio-Parts.pretty-master:SK6812-MINI-E, B.Cu at (313.1, 109.1)
- added D101: LED_SK6812MINI, Keebio-Parts.pretty-master:SK6812-MINI-E, B.Cu at (332.2, 111.1)
- added D102: LED_SK6812MINI, Keebio-Parts.pretty-master:SK6812-MINI-E, B.Cu at (351.2, 116.1)
- added D103: LED_SK6812MINI, Keebio-Parts.pretty-master:SK6812-MINI-E, B.Cu at (370.3, 119.1)
- added D104: LED_SK6812MINI, Keebio-Parts.pretty-master:SK6812-MINI-E, B.Cu at (275.0, 133.1)
- added D105: LED_SK6812MINI, Keebio-Parts.pretty-master:SK6812-MINI-E, B.Cu at (294.1, 130.1)
- added D106: LED_SK6812MINI, Keebio-Parts.pretty-master:SK6812-MINI-E, B.Cu at (313.1, 128.1)
- added D107: LED_SK6812MINI, Keebio-Parts.pretty-master:SK6812-MINI-E, B.Cu at (332.2, 130.1)
- added D108: LED_SK6812MINI, Keebio-Parts.pretty-master:SK6812-MINI-E, B.Cu at (351.2, 135.1)
- added D109: LED_SK6812MINI, Keebio-Parts.pretty-master:SK6812-MINI-E, B.Cu at (370.3, 138.1)
- added D11: Diode, ScottoKeebs_Components:Diode_SOD-123, B.Cu at (101.1, 97.6)
- added D110: LED_SK6812MINI, Keebio-Parts.pretty-master:SK6812-MINI-E, B.Cu at (275.0, 152.2)
- added D111: LED_SK6812MINI, Keebio-Parts.pretty-master:SK6812-MINI-E, B.Cu at (294.1, 149.2)
- added D112: LED_SK6812MINI, Keebio-Parts.pretty-master:SK6812-MINI-E, B.Cu at (313.1, 147.2)
- added D113: LED_SK6812MINI, Keebio-Parts.pretty-master:SK6812-MINI-E, B.Cu at (332.2, 149.2)
- added D114: LED_SK6812MINI, Keebio-Parts.pretty-master:SK6812-MINI-E, B.Cu at (351.2, 154.2)
- added D115: LED_SK6812MINI, Keebio-Parts.pretty-master:SK6812-MINI-E, B.Cu at (370.3, 157.2)
- added D116: LED_SK6812MINI, Keebio-Parts.pretty-master:SK6812-MINI-E, B.Cu at (256.0, 142.7)
- added D117: LED_SK6812MINI, Keebio-Parts.pretty-master:SK6812-MINI-E, B.Cu at (255.0, 168.9)
- added D118: LED_SK6812MINI, Keebio-Parts.pretty-master:SK6812-MINI-E, B.Cu at (284.6, 171.2)
- added D119: LED_SK6812MINI, Keebio-Parts.pretty-master:SK6812-MINI-E, B.Cu at (303.6, 168.2)
- added D12: Diode, ScottoKeebs_Components:Diode_SOD-123, B.Cu at (100.8, 133.2)
- added D120: LED_SK6812MINI, Keebio-Parts.pretty-master:SK6812-MINI-E, B.Cu at (322.7, 168.2)
- added D13: Diode, ScottoKeebs_Components:Diode_SOD-123, B.Cu at (101.2, 135.7)
- added D14: Diode, ScottoKeebs_Components:Diode_SOD-123, B.Cu at (129.8, 154.5)
- added D15: Diode, ScottoKeebs_Components:Diode_SOD-123, B.Cu at (120.2, 92.5)
- added D16: Diode, ScottoKeebs_Components:Diode_SOD-123, B.Cu at (120.2, 95.5)
- added D17: Diode, ScottoKeebs_Components:Diode_SOD-123, B.Cu at (119.7, 131.2)
- added D18: Diode, ScottoKeebs_Components:Diode_SOD-123, B.Cu at (119.2, 133.6)
- added D19: Diode, ScottoKeebs_Components:Diode_SOD-123, B.Cu at (148.9, 157.9)
- added D2: Diode, ScottoKeebs_Components:Diode_SOD-123, B.Cu at (63.1, 105.6)
- added D20: Diode, ScottoKeebs_Components:Diode_SOD-123, B.Cu at (139.3, 94.3)
- added D21: Diode, ScottoKeebs_Components:Diode_SOD-123, B.Cu at (139.3, 97.6)
- added D22: Diode, ScottoKeebs_Components:Diode_SOD-123, B.Cu at (139.9, 133.0)
- added D23: Diode, ScottoKeebs_Components:Diode_SOD-123, B.Cu at (140.0, 136.0)
- added D24: Diode, ScottoKeebs_Components:Diode_SOD-123, B.Cu at (164.3, 153.9)
- added D25: Diode, ScottoKeebs_Components:Diode_SOD-123, B.Cu at (158.3, 97.3)
- added D26: Diode, ScottoKeebs_Components:Diode_SOD-123, B.Cu at (158.3, 100.3)
- added D27: Diode, ScottoKeebs_Components:Diode_SOD-123, B.Cu at (158.3, 135.4)
- added D28: Diode, ScottoKeebs_Components:Diode_SOD-123, B.Cu at (158.3, 155.7)
- added D29: Diode, ScottoKeebs_Components:Diode_SOD-123, B.Cu at (168.5, 127.1)
- added D3: Diode, ScottoKeebs_Components:Diode_SOD-123, B.Cu at (63.1, 140.6)
- added D30: Diode, ScottoKeebs_Components:Diode_SOD-123, B.Cu at (192.7, 106.9)
- added D31: Diode, ScottoKeebs_Components:Diode_SOD-123, B.Cu at (192.7, 103.6)
- added D32: Diode, ScottoKeebs_Components:Diode_SOD-123, B.Cu at (192.7, 100.2)
- added D33: Diode, ScottoKeebs_Components:Diode_SOD-123, B.Cu at (189.2, 95.4)
- added D34: LED_SK6812MINI, Keebio-Parts.pretty-master:SK6812-MINI-E, B.Cu at (151.2, 95.0)
- added D35: LED_SK6812MINI, Keebio-Parts.pretty-master:SK6812-MINI-E, B.Cu at (132.2, 92.0)
- added D36: LED_SK6812MINI, Keebio-Parts.pretty-master:SK6812-MINI-E, B.Cu at (113.1, 90.0)
- added D37: LED_SK6812MINI, Keebio-Parts.pretty-master:SK6812-MINI-E, B.Cu at (94.1, 92.0)
- added D38: LED_SK6812MINI, Keebio-Parts.pretty-master:SK6812-MINI-E, B.Cu at (75.0, 97.0)
- added D39: LED_SK6812MINI, Keebio-Parts.pretty-master:SK6812-MINI-E, B.Cu at (56.0, 100.0)
- added D4: Diode, ScottoKeebs_Components:Diode_SOD-123, B.Cu at (63.1, 143.7)
- added D40: LED_SK6812MINI, Keebio-Parts.pretty-master:SK6812-MINI-E, B.Cu at (151.2, 114.1)
- added D41: LED_SK6812MINI, Keebio-Parts.pretty-master:SK6812-MINI-E, B.Cu at (132.2, 111.1)
- added D42: LED_SK6812MINI, Keebio-Parts.pretty-master:SK6812-MINI-E, B.Cu at (113.1, 109.1)
- added D43: LED_SK6812MINI, Keebio-Parts.pretty-master:SK6812-MINI-E, B.Cu at (94.1, 111.1)
- added D44: LED_SK6812MINI, Keebio-Parts.pretty-master:SK6812-MINI-E, B.Cu at (75.0, 116.1)
- added D45: LED_SK6812MINI, Keebio-Parts.pretty-master:SK6812-MINI-E, B.Cu at (56.0, 119.1)
- added D46: LED_SK6812MINI, Keebio-Parts.pretty-master:SK6812-MINI-E, B.Cu at (151.2, 133.1)
- added D47: LED_SK6812MINI, Keebio-Parts.pretty-master:SK6812-MINI-E, B.Cu at (132.2, 130.1)
- added D48: LED_SK6812MINI, Keebio-Parts.pretty-master:SK6812-MINI-E, B.Cu at (113.1, 128.1)
- added D49: LED_SK6812MINI, Keebio-Parts.pretty-master:SK6812-MINI-E, B.Cu at (94.1, 130.1)
- added D5: Diode, ScottoKeebs_Components:Diode_SOD-123, B.Cu at (82.1, 99.7)
- added D50: LED_SK6812MINI, Keebio-Parts.pretty-master:SK6812-MINI-E, B.Cu at (75.0, 135.1)
- added D51: LED_SK6812MINI, Keebio-Parts.pretty-master:SK6812-MINI-E, B.Cu at (56.0, 138.1)
- added D52: LED_SK6812MINI, Keebio-Parts.pretty-master:SK6812-MINI-E, B.Cu at (151.2, 152.2)
- added D53: LED_SK6812MINI, Keebio-Parts.pretty-master:SK6812-MINI-E, B.Cu at (132.2, 149.2)
- added D54: LED_SK6812MINI, Keebio-Parts.pretty-master:SK6812-MINI-E, B.Cu at (113.1, 147.2)
- added D55: LED_SK6812MINI, Keebio-Parts.pretty-master:SK6812-MINI-E, B.Cu at (94.1, 149.2)
- added D56: LED_SK6812MINI, Keebio-Parts.pretty-master:SK6812-MINI-E, B.Cu at (75.0, 154.2)
- added D57: LED_SK6812MINI, Keebio-Parts.pretty-master:SK6812-MINI-E, B.Cu at (56.0, 157.2)
- added D58: LED_SK6812MINI, Keebio-Parts.pretty-master:SK6812-MINI-E, B.Cu at (170.3, 142.7)
- added D59: LED_SK6812MINI, Keebio-Parts.pretty-master:SK6812-MINI-E, B.Cu at (171.2, 168.9)
- added D6: Diode, ScottoKeebs_Components:Diode_SOD-123, B.Cu at (82.1, 102.7)
- added D60: LED_SK6812MINI, Keebio-Parts.pretty-master:SK6812-MINI-E, B.Cu at (141.7, 171.2)
- added D61: LED_SK6812MINI, Keebio-Parts.pretty-master:SK6812-MINI-E, B.Cu at (122.6, 168.2)
- added D62: LED_SK6812MINI, Keebio-Parts.pretty-master:SK6812-MINI-E, B.Cu at (103.6, 168.2)
- added D63: Diode, ScottoKeebs_Components:Diode_SOD-123, B.Cu at (282.3, 98.5)
- added D64: Diode, ScottoKeebs_Components:Diode_SOD-123, B.Cu at (282.3, 100.9)
- added D65: Diode, ScottoKeebs_Components:Diode_SOD-123, B.Cu at (282.2, 136.0)
- added D66: Diode, ScottoKeebs_Components:Diode_SOD-123, B.Cu at (225.8, 125.4)
- added D67: Diode, ScottoKeebs_Components:Diode_SOD-123, B.Cu at (225.8, 122.0)
- added D68: Diode, ScottoKeebs_Components:Diode_SOD-123, B.Cu at (225.8, 118.7)
- added D69: Diode, ScottoKeebs_Components:Diode_SOD-123, B.Cu at (225.8, 115.3)
- added D7: Diode, ScottoKeebs_Components:Diode_SOD-123, B.Cu at (82.1, 137.6)
- added D70: Diode, ScottoKeebs_Components:Diode_SOD-123, B.Cu at (301.4, 133.6)
- added D71: Diode, ScottoKeebs_Components:Diode_SOD-123, B.Cu at (300.8, 136.0)
- added D72: Diode, ScottoKeebs_Components:Diode_SOD-123, B.Cu at (262.1, 155.7)
- added D73: Diode, ScottoKeebs_Components:Diode_SOD-123, B.Cu at (320.4, 92.5)
- added D74: Diode, ScottoKeebs_Components:Diode_SOD-123, B.Cu at (320.4, 95.5)
- added D75: Diode, ScottoKeebs_Components:Diode_SOD-123, B.Cu at (231.5, 125.4)
- added D76: Diode, ScottoKeebs_Components:Diode_SOD-123, B.Cu at (231.5, 122.0)
- added D77: Diode, ScottoKeebs_Components:Diode_SOD-123, B.Cu at (231.5, 118.7)
- added D78: Diode, ScottoKeebs_Components:Diode_SOD-123, B.Cu at (231.5, 115.3)
- added D79: Diode, ScottoKeebs_Components:Diode_SOD-123, B.Cu at (231.5, 112.0)
- added D8: Diode, ScottoKeebs_Components:Diode_SOD-123, B.Cu at (82.1, 141.1)
- added D80: Diode, ScottoKeebs_Components:Diode_SOD-123, B.Cu at (231.5, 108.6)
- added D81: Diode, ScottoKeebs_Components:Diode_SOD-123, B.Cu at (231.5, 105.3)
- added D82: Diode, ScottoKeebs_Components:Diode_SOD-123, B.Cu at (231.5, 101.9)
- added D83: Diode, ScottoKeebs_Components:Diode_SOD-123, B.Cu at (357.9, 100.3)
- added D84: Diode, ScottoKeebs_Components:Diode_SOD-123, B.Cu at (237.3, 125.4)
- added D85: Diode, ScottoKeebs_Components:Diode_SOD-123, B.Cu at (237.3, 122.0)
- added D86: Diode, ScottoKeebs_Components:Diode_SOD-123, B.Cu at (237.3, 118.7)
- added D87: Diode, ScottoKeebs_Components:Diode_SOD-123, B.Cu at (237.3, 115.3)
- added D88: Diode, ScottoKeebs_Components:Diode_SOD-123, B.Cu at (237.3, 112.0)
- added D89: Diode, ScottoKeebs_Components:Diode_SOD-123, B.Cu at (237.3, 108.6)
- added D9: Diode, ScottoKeebs_Components:Diode_SOD-123, B.Cu at (110.9, 154.7)
- added D90: Diode, ScottoKeebs_Components:Diode_SOD-123, B.Cu at (237.3, 105.3)
- added D91: Diode, ScottoKeebs_Components:Diode_SOD-123, B.Cu at (237.3, 101.9)
- added D92: LED_SK6812MINI, Keebio-Parts.pretty-master:SK6812-MINI-E, B.Cu at (275.0, 95.0)
- added D93: LED_SK6812MINI, Keebio-Parts.pretty-master:SK6812-MINI-E, B.Cu at (294.1, 92.0)
- added D94: LED_SK6812MINI, Keebio-Parts.pretty-master:SK6812-MINI-E, B.Cu at (313.1, 90.0)
- added D95: LED_SK6812MINI, Keebio-Parts.pretty-master:SK6812-MINI-E, B.Cu at (332.2, 92.0)
- added D96: LED_SK6812MINI, Keebio-Parts.pretty-master:SK6812-MINI-E, B.Cu at (351.2, 97.0)
- added D97: LED_SK6812MINI, Keebio-Parts.pretty-master:SK6812-MINI-E, B.Cu at (370.3, 100.0)
- added D98: LED_SK6812MINI, Keebio-Parts.pretty-master:SK6812-MINI-E, B.Cu at (275.0, 114.1)
- added D99: LED_SK6812MINI, Keebio-Parts.pretty-master:SK6812-MINI-E, B.Cu at (294.1, 111.1)
- added E1: TSWB3NCB111LFS, ANO_Encoder:Encoder_TSWB3NCB111LFS, F.Cu at (207.7, 155.7)
- added J3: Conn_01x10_Socket, Connector_FFC-FPC:Hirose_FH12-10S-0.5SH_1x10-1MP_P0.50mm_Horizontal, B.Cu at (173.2, 152.4)
- added J4: Conn_01x10_Pin, Connector_FFC-FPC:Hirose_FH12-10S-0.5SH_1x10-1MP_P0.50mm_Horizontal, B.Cu at (199.4, 148.2)
- added SW1: SW_SPDT, SSSS811101:SW_SSSS811101, B.Cu at (180.4, 119.1)
- added SW2: SW_Push, ul_EVQ-PUJ02K:SW_EVQPUJ_4P7X3P5_PAN, B.Cu at (179.8, 128.1)
- added SW3: SW_SPDT, SSSS811101:SW_SSSS811101, B.Cu at (245.9, 118.8)
- added SW4: SW_Push, ul_EVQ-PUJ02K:SW_EVQPUJ_4P7X3P5_PAN, B.Cu at (246.5, 127.5)
- S1: renamed from S4; value (none) -> Keyswitch
- S10: renamed from S12; value (none) -> Keyswitch
- S11, S20: value (none) -> Keyswitch
- S12: renamed from S10; value (none) -> Keyswitch
- S13: renamed from S9; value (none) -> Keyswitch
- S14: renamed from S27; value (none) -> Keyswitch
- S15: renamed from S16; value (none) -> Keyswitch
- S16: renamed from S15; value (none) -> Keyswitch
- S17: renamed from S14; value (none) -> Keyswitch
- S18: renamed from S13; value (none) -> Keyswitch
- S19: renamed from S28; value (none) -> Keyswitch
- S2: renamed from S3; value (none) -> Keyswitch
- S21: renamed from S19; value (none) -> Keyswitch
- S22: renamed from S18; value (none) -> Keyswitch
- S23: renamed from S17; value (none) -> Keyswitch
- S24: renamed from S29; value (none) -> Keyswitch
- S25: renamed from S24; value (none) -> Keyswitch
- S26: renamed from S23; value (none) -> Keyswitch
- S27: renamed from S22; value (none) -> Keyswitch
- S28: renamed from S21; value (none) -> Keyswitch
- S29: renamed from S25; value (none) -> Keyswitch
- S3: renamed from S2; value (none) -> Keyswitch
- S30: renamed from S53; value (none) -> Keyswitch
- S31: renamed from S52; value (none) -> Keyswitch
- S32: renamed from S51; value (none) -> Keyswitch
- S33: renamed from S50; value (none) -> Keyswitch
- S34: renamed from S54; value (none) -> Keyswitch
- S35: renamed from S49; value (none) -> Keyswitch
- S36: renamed from S48; value (none) -> Keyswitch
- S37: renamed from S47; value (none) -> Keyswitch
- S38: renamed from S46; value (none) -> Keyswitch
- S39: renamed from S58; value (none) -> Keyswitch
- S4: renamed from S1; value (none) -> Keyswitch
- S40: renamed from S45; value (none) -> Keyswitch
- S41: renamed from S44; value (none) -> Keyswitch
- S42: renamed from S43; value (none) -> Keyswitch
- S43: renamed from S42; value (none) -> Keyswitch
- S44: renamed from S57; value (none) -> Keyswitch
- S45: renamed from S41; value (none) -> Keyswitch
- S46: renamed from S40; value (none) -> Keyswitch
- S47: renamed from S39; value (none) -> Keyswitch
- S48: renamed from S38; value (none) -> Keyswitch
- S49: renamed from S56; value (none) -> Keyswitch
- S5: renamed from S8; value (none) -> Keyswitch
- S50: renamed from S37; value (none) -> Keyswitch
- S51: renamed from S36; value (none) -> Keyswitch
- S52: renamed from S35; value (none) -> Keyswitch
- S53: renamed from S34; value (none) -> Keyswitch
- S54: renamed from S55; value (none) -> Keyswitch
- S55: renamed from S33; value (none) -> Keyswitch
- S56: renamed from S32; value (none) -> Keyswitch
- S57: renamed from S31; value (none) -> Keyswitch
- S58: renamed from S30; value (none) -> Keyswitch
- S6: renamed from S7; value (none) -> Keyswitch
- S7: renamed from S6; value (none) -> Keyswitch
- S8: renamed from S5; value (none) -> Keyswitch
- S9: renamed from S26; value (none) -> Keyswitch
- renumbered U4 to U1, U1 to U2
Connections:
- S1 pad 1: (no net) -> L-COL0
- S1 pad 2: outer_stretch -> Net-(D1-A)
- S10 pad 1: (no net) -> L-COL2
- S10 pad 2: ring_stretch -> Net-(D10-A)
- S11 pad 1: (no net) -> L-COL2
- S11 pad 2: ring_top -> Net-(D11-A)
- S12 pad 1: (no net) -> L-COL2
- S12 pad 2: ring_home -> Net-(D12-A)
- S13 pad 1: (no net) -> L-COL2
- S13 pad 2: ring_bottom -> Net-(D13-A)
- S14 pad 1: (no net) -> L-COL2
- S14 pad 2: tucky2_stretch -> Net-(D14-A)
- S15 pad 1: (no net) -> L-COL3
- S15 pad 2: middle_stretch -> Net-(D15-A)
- S16 pad 1: (no net) -> L-COL3
- S16 pad 2: middle_top -> Net-(D16-A)
- S17 pad 1: (no net) -> L-COL3
- S17 pad 2: middle_home -> Net-(D17-A)
- S18 pad 1: (no net) -> L-COL3
- S18 pad 2: middle_bottom -> Net-(D18-A)
- S19 pad 1: (no net) -> L-COL3
- S19 pad 2: tucky3_stretch -> Net-(D19-A)
- S2 pad 1: (no net) -> L-COL0
- S2 pad 2: outer_top -> Net-(D2-A)
- S20 pad 1: (no net) -> L-COL4
- S20 pad 2: index_stretch -> Net-(D20-A)
- S21 pad 1: (no net) -> L-COL4
- S21 pad 2: index_top -> Net-(D21-A)
- S22 pad 1: (no net) -> L-COL4
- S22 pad 2: index_home -> Net-(D22-A)
- S23 pad 1: (no net) -> L-COL4
- S23 pad 2: index_bottom -> Net-(D23-A)
- S24 pad 1: (no net) -> L-COL4
- S24 pad 2: reachy_stretch -> Net-(D24-A)
- S25 pad 1: (no net) -> L-COL5
- S25 pad 2: inner_stretch -> Net-(D25-A)
- S26 pad 1: (no net) -> L-COL5
- S26 pad 2: inner_top -> Net-(D26-A)
- S27 pad 1: (no net) -> L-COL5
- S27 pad 2: inner_home -> Net-(D27-A)
- S28 pad 1: (no net) -> L-COL5
- S28 pad 2: inner_bottom -> Net-(D28-A)
- S29 pad 1: (no net) -> L-COL5
- S29 pad 2: reach_reach -> Net-(D29-A)
- S3 pad 1: (no net) -> L-COL0
- S3 pad 2: outer_home -> Net-(D3-A)
- S30 pad 1: (no net) -> R-COL5
- S30 pad 2: mirror_inner_stretch -> Net-(D63-A)
- S31 pad 1: (no net) -> R-COL5
- S31 pad 2: mirror_inner_top -> Net-(D64-A)
- S32 pad 1: (no net) -> R-COL5
- S32 pad 2: mirror_inner_home -> Net-(D65-A)
- S33 pad 1: (no net) -> R-COL5
- S33 pad 2: mirror_inner_bottom -> Net-(D66-A)
- S34 pad 1: (no net) -> R-COL5
- S34 pad 2: mirror_reach_reach -> Net-(D67-A)
- S35 pad 1: (no net) -> R-COL4
- S35 pad 2: mirror_index_stretch -> Net-(D68-A)
- S36 pad 1: (no net) -> R-COL4
- S36 pad 2: mirror_index_top -> Net-(D69-A)
- S37 pad 1: (no net) -> R-COL4
- S37 pad 2: mirror_index_home -> Net-(D70-A)
- S38 pad 1: (no net) -> R-COL4
- S38 pad 2: mirror_index_bottom -> Net-(D71-A)
- S39 pad 1: (no net) -> R-COL4
- S39 pad 2: mirror_reachy_stretch -> Net-(D72-A)
- S4 pad 1: (no net) -> L-COL0
- S4 pad 2: outer_bottom -> Net-(D4-A)
- S40 pad 1: (no net) -> R-COL3
- S40 pad 2: mirror_middle_stretch -> Net-(D73-A)
- S41 pad 1: (no net) -> R-COL3
- S41 pad 2: mirror_middle_top -> Net-(D74-A)
- S42 pad 1: (no net) -> R-COL3
- S42 pad 2: mirror_middle_home -> Net-(D75-A)
- S43 pad 1: (no net) -> R-COL3
- S43 pad 2: mirror_middle_bottom -> Net-(D76-A)
- S44 pad 1: (no net) -> R-COL3
- S44 pad 2: mirror_tucky3_stretch -> Net-(D77-A)
- S45 pad 1: (no net) -> R-COL2
- S45 pad 2: mirror_ring_stretch -> Net-(D78-A)
- S46 pad 1: (no net) -> R-COL2
- S46 pad 2: mirror_ring_top -> Net-(D79-A)
- S47 pad 1: (no net) -> R-COL2
- S47 pad 2: mirror_ring_home -> Net-(D80-A)
- S48 pad 1: (no net) -> R-COL2
- S48 pad 2: mirror_ring_bottom -> Net-(D81-A)
- S49 pad 1: (no net) -> R-COL2
- S49 pad 2: mirror_tucky2_stretch -> Net-(D82-A)
- S5 pad 1: (no net) -> L-COL1
- S5 pad 2: pinky_stretch -> Net-(D5-A)
- S50 pad 1: (no net) -> R-COL1
- S50 pad 2: mirror_pinky_stretch -> Net-(D83-A)
- S51 pad 1: (no net) -> R-COL1
- S51 pad 2: mirror_pinky_top -> Net-(D84-A)
- S52 pad 1: (no net) -> R-COL1
- S52 pad 2: mirror_pinky_home -> Net-(D85-A)
- S53 pad 1: (no net) -> R-COL1
- S53 pad 2: mirror_pinky_bottom -> Net-(D86-A)
- S54 pad 1: (no net) -> R-COL1
- S54 pad 2: mirror_tucky1_stretch -> Net-(D87-A)
- S55 pad 1: (no net) -> R-COL0
- S55 pad 2: mirror_outer_stretch -> Net-(D88-A)
- S56 pad 1: (no net) -> R-COL0
- S56 pad 2: mirror_outer_top -> Net-(D89-A)
- S57 pad 1: (no net) -> R-COL0
- S57 pad 2: mirror_outer_home -> Net-(D90-A)
- S58 pad 1: (no net) -> R-COL0
- S58 pad 2: mirror_outer_bottom -> Net-(D91-A)
- S6 pad 1: (no net) -> L-COL1
- S6 pad 2: pinky_top -> Net-(D6-A)
- S7 pad 1: (no net) -> L-COL1
- S7 pad 2: pinky_home -> Net-(D7-A)
- S8 pad 1: (no net) -> L-COL1
- S8 pad 2: pinky_bottom -> Net-(D8-A)
- S9 pad 1: (no net) -> L-COL1
- S9 pad 2: tucky1_stretch -> Net-(D9-A)
- U1 pad 18: L-COL6 -> COMB
Routing:
- net GND: track 0.00 -> 570.7 mm, vias 0 -> 29
- net +3V3: track 0.00 -> 439.4 mm, vias 0 -> 29
- net L-ROW1: track 0.00 -> 110.7 mm
- net L-ROW0: track 0.00 -> 110.3 mm
- net L-COL1: track 0.00 -> 79.4 mm, vias 0 -> 4
- net L-COL0: track 0.00 -> 76.6 mm, vias 0 -> 4
- net L-ROW2: track 0.00 -> 69.9 mm
- net L-COL4: track 0.00 -> 61.5 mm, vias 0 -> 4
- net Net-(D40-DOUT): track 0.00 -> 34.3 mm
- net Net-(D37-DOUT): track 0.00 -> 33.5 mm
- net Net-(D39-DOUT): track 0.00 -> 33.3 mm
- net Net-(D51-DOUT): track 0.00 -> 33.3 mm
- net Net-(D58-DOUT): track 0.00 -> 32.9 mm
- net Net-(D49-DOUT): track 0.00 -> 32.7 mm
- net Net-(D50-DOUT): track 0.00 -> 31.2 mm
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
Commit message: updates to pcb
Parts:
- SW1, SW2, SW3, SW4: moved to F.Cu
- moved J4 104.1 mm to (109.5, 200.6)
- moved E1 101.6 mm to (118.5, 204.5)
- moved D28 16.7 mm to (158.3, 139.0)
- moved D29 3.61 mm to (164.9, 127.7), turned to 180 degrees
- moved BT1 3.28 mm to (171.0, 88.2)
- moved D24 2.15 mm to (163.1, 155.7)
- moved D18 1.15 mm to (120.2, 134.1)
- moved D22 0.82 mm to (139.3, 132.4)
- moved SW3 0.77 mm to (246.5, 119.3), turned to -90 degrees
- moved D23 0.71 mm to (139.3, 136.0)
- moved D17 0.67 mm to (120.2, 130.9)
- moved J1 0.66 mm to (165.0, 118.5)
- moved SW1 0.62 mm to (179.8, 119.3), turned to 90 degrees
- moved Display1 0.56 mm to (171.1, 98.4)
- moved U1 0.52 mm to (171.1, 98.2)
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Routing:
- net GND: track 570.7 -> 837.1 mm
- net +3V3: track 439.4 -> 690.8 mm, vias 29 -> 30
- net L-COL2: track 15.1 -> 196.5 mm, vias 1 -> 5
- net L-COL3: track 10.0 -> 188.3 mm, vias 1 -> 5
- net L-COL1: track 79.4 -> 215.8 mm, vias 4 -> 5
- net L-COL0: track 76.6 -> 189.5 mm
- net L-ROW3: track 21.3 -> 134.1 mm
- net L-COL4: track 61.5 -> 170.2 mm, vias 4 -> 5
- net L-ROW4: track 0.00 -> 103.9 mm, vias 0 -> 2
- net L-COL5: track 5.02 -> 83.0 mm, vias 1 -> 4
- net L-ROW2: track 69.9 -> 135.8 mm
- net Net-(D59-DOUT): track 0.00 -> 38.5 mm
- net Net-(D48-DOUT): track 0.00 -> 30.5 mm
- net Net-(D60-DOUT): track 0.00 -> 30.5 mm
- net Net-(D47-DOUT): track 0.00 -> 29.7 mm
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Other:
- board size 334.4 x 109.5 mm -> 334.4 x 147.7 mm

Commit message: todays progress
Parts:
- S1, S10, S11, S12, S13, S14, S15, S16, S17, S18, S19, S2, S20, S21, S22, S23, S24, S25, S26, S27, S28, S29, S3, S30, S31, S32, S33, S34, S35, S36, S37, S38, S39, S4, S40, S41, S42, S43, S44, S45, S46, S47, S48, S49, S5, S50, S51, S52, S53, S54, S55, S56, S57, S58, S6, S7, S8, S9: footprint comboswitch:Hotswap_Choc_V1V2 -> Hotswap_Choc_and_MX:Hotswap_Choc_V1V2
Routing:
- net GND: track 837.1 -> 791.8 mm
- net +3V3: track 690.8 -> 701.9 mm, vias 30 -> 29
- net L-COL0: track 189.5 -> 182.5 mm
- net L-COL2: track 196.5 -> 202.4 mm
- net L-COL1: track 215.8 -> 221.4 mm
- net Net-(D10-A): track 12.4 -> 15.4 mm
- net Net-(D9-A): track 8.53 -> 6.17 mm
- net Net-(D3-A): track 15.5 -> 16.7 mm
- net Net-(D1-A): track 15.2 -> 16.2 mm
- net Net-(D22-A): track 15.5 -> 16.2 mm
- net Net-(D20-A): track 15.5 -> 16.2 mm
- net Net-(D7-A): track 15.6 -> 16.3 mm
- net Net-(D5-A): track 16.2 -> 16.9 mm
- net Net-(D15-A): track 15.7 -> 16.4 mm
- net Net-(D17-A): track 16.0 -> 16.7 mm
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