File: PCB/quartz58.kicad_pcb (KiCad board)
At the start: 2 copper layers, 334.4 x 147.7 mm, 193 parts, among them J1 OLED_128x32, J2 OLED_128x32, J3 Conn_01x10_Socket, J4 Conn_01x10_Pin, SW1 SW_SPDT, SW2 SW_Push, SW3 SW_SPDT, SW4 SW_Push, U1 Nice_Nano_V2, U2 Nice_Nano_V2

Commit message: might be cooked chat
Parts:
- added REF**: Encoder_TSWB3NCB111LFS_Breakout, ANO_Encoder:Encoder_TSWB3NCB111LFS_Breakout, F.Cu at (179.4, 136.4)
- moved D91 146.2 mm to (377.4, 143.5)
- moved D90 144.5 mm to (377.4, 140.6)
- moved D88 140.5 mm to (377.4, 102.5)
- moved D89 140.2 mm to (377.4, 105.4)
- moved D84 123.3 mm to (358.4, 102.5)
- moved D86 123.1 mm to (358.4, 140.6)
- moved D85 122.1 mm to (358.4, 137.6)
- moved D81 112.1 mm to (339.3, 135.8)
- moved D80 110.5 mm to (339.3, 132.8)
- moved D78 109.8 mm to (339.3, 94.7)
- moved D79 108.8 mm to (339.3, 97.7)
- moved D87 100.9 mm to (329.8, 155.4)
- moved D82 95.6 mm to (310.7, 155.4)
- moved D76 89.6 mm to (320.3, 134.0)
- moved D75 88.9 mm to (320.3, 131.0)
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Connections:
- SW2 pad 1: GND -> L-RST
- SW2 pad 2: L-RST -> GND
- SW4 pad 1: GND -> R-RST
- SW4 pad 2: R-RST -> GND
- U1 pad 1: L-ENCODER-A0 -> L-ENCODER-B0
- U1 pad 2: L-ENCODER-B0 -> L-ENCODER-A0
Routing:
- net GND: track 791.8 -> 926.9 mm, vias 29 -> 30
- net R-ROW0: track 0.00 -> 122.2 mm
- net R-ROW1: track 0.00 -> 104.2 mm
- net R-ROW2: track 0.00 -> 83.1 mm
- net R-ROW3: track 0.00 -> 82.2 mm
- net L-ENCODER-B0: track 0.00 -> 78.6 mm
- net L-ENCODER-A0: track 0.00 -> 76.0 mm
- net R-ROW4: track 0.00 -> 70.2 mm
- net +3V3: track 701.9 -> 767.8 mm, vias 29 -> 28
- net L-COL5: track 83.0 -> 145.1 mm
- net L-ROW0: track 110.3 -> 172.1 mm, vias 0 -> 1
- net L-ROW1: track 111.4 -> 169.2 mm, vias 0 -> 1
- net SW1: track 0.00 -> 55.1 mm, vias 0 -> 1
- net Net-(SW1-B): track 0.00 -> 48.7 mm
- net L-COL0: track 182.5 -> 230.6 mm
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Other:
- board size 334.4 x 147.7 mm -> 334.4 x 146.4 mm

Commit message: todays progress
Parts:
- moved J4 1.40 mm to (126.3, 200.2)
- turned E1 to 180 degrees
Connections:
- J4 pad 1: Net-(E1-ENCA) -> unconnected-(J4-Pin_1-Pad1)
- J4 pad 10: unconnected-(J4-Pin_10-Pad10) -> Net-(E1-ENCA)
- J4 pad 2: Net-(E1-ENCB) -> Net-(E1-COMB)
- J4 pad 3: Net-(E1-COMA) -> Net-(E1-SW5)
- J4 pad 4: Net-(E1-SW1) -> Net-(E1-SW4)
- J4 pad 5: Net-(E1-SW2) -> Net-(E1-SW3)
- J4 pad 6: Net-(E1-SW3) -> Net-(E1-SW2)
- J4 pad 7: Net-(E1-SW4) -> Net-(E1-SW1)
- J4 pad 8: Net-(E1-SW5) -> Net-(E1-COMA)
- J4 pad 9: Net-(E1-COMB) -> Net-(E1-ENCB)
Routing:
- net Net-(E1-SW3): track 35.3 -> 11.5 mm
- net Net-(E1-SW5): track 7.08 -> 29.5 mm
- net Net-(E1-ENCA): track 22.5 -> 6.91 mm, vias 0 -> 1
- net Net-(E1-COMA): track 7.68 -> 22.7 mm, vias 0 -> 1
- net Net-(E1-SW2): track 26.2 -> 11.8 mm
- net Net-(E1-SW4): track 17.1 -> 26.7 mm
- net Net-(E1-ENCB): track 20.7 -> 13.3 mm, vias 0 -> 1
- net Net-(E1-COMB): track 22.1 -> 18.1 mm
- net Net-(E1-SW1): track 11.4 -> 13.4 mm, vias 0 -> 1
Other:
- board size 334.4 x 146.4 mm -> 334.4 x 146.3 mm

Commit message: more progress
Parts:
- moved U1 1.47 mm to (170.3, 99.4)
- moved Display1 1.27 mm to (170.3, 99.4)
- moved J1 1.07 mm to (164.3, 119.3)
- moved U2 0.89 mm to (256.0, 99.3)
- moved Display2 0.69 mm to (256.0, 99.3)
- moved J2 0.11 mm to (250.0, 119.2)
Changed lines of the file:
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@@
 		(allow_soldermask_bridges_in_footprints no)
 		(tenting front back)
-		(grid_origin 135.539381 202.781752)
+		(grid_origin 255.976607 99.277544)
 		(pcbplotparams
 			(layerselection 0x00000000_00000000_55555555_5755f5ff)
@@
 	(footprint "ScottoKeebs_Components:OLED_128x32"
 		(layer "F.Cu")
-		(at 249.915128 119.075722 90)
+		(at 249.976607 119.167544 90)
 		(property "Reference" "J2"
 			(at 7.75 10 90)
@@
 	(footprint "nice_view:nice_view"
 		(layer "F.Cu")
-		(at 255.984502 98.58447)
+		(at 255.976607 99.277544)
 		(property "Reference" "Display2"
 			(at 0 1.27 0)
@@
 	(footprint "nice_view:nice_view"
 		(layer "F.Cu")
-		(at 171.086607 98.417544)
+		(at 170.251607 99.377544)
 		(property "Reference" "Display1"
 			(at 0 1.27 0)
@@
 	(footprint "ScottoKeebs_Components:OLED_128x32"
 		(layer "F.Cu")
-		(at 165.026607 118.527544 90)
+		(at 164.251607 119.267544 90)
 		(property "Reference" "J1"
 			(at 7.75 10 90)
@@
 	(footprint "nice-nano-kicad-master:nice_nano"
 		(layer "B.Cu")
-		(at 256.131607 98.397544 -90)
+		(at 255.976607 99.277544 -90)
 		(property "Reference" "U2"
 			(at 0 -1.625 90)
@@
 	(footprint "nice-nano-kicad-master:nice_nano"
 		(layer "B.Cu")
-		(at 171.346607 98.397544 -90)
+		(at 170.251607 99.377544 -90)
 		(property "Reference" "U1"
 			(at 0 -1.625 90)

Commit message: left side ready for review
Parts:
- added REF**: Display Cover Mounting Holes, Display_Cover_Mounting_Holes:for_nice_nano, F.Cu at (170.3, 97.6)
- added REF**: Display Cover Mounting Holes, Display_Cover_Mounting_Holes:for_nice_nano, B.Cu at (255.9, 101.0)
- moved SW2 8.85 mm to (179.7, 117.7)
- moved SW1 7.45 mm to (179.9, 125.9)
- moved BT1 3.65 mm to (170.3, 87.4)
- moved BT2 1.34 mm to (256.0, 87.3)
- moved J2 0.76 mm to (250.0, 119.9)
- moved J1 0.66 mm to (164.3, 119.9)
- moved D24 0.42 mm to (163.1, 156.1)
- moved SW4 0.23 mm to (246.5, 127.2)
- moved SW3 0.20 mm to (246.5, 119.1)
Connections:
- net Net-(SW3-B) renamed +3V8
- S30 pad 1: R-COL5 -> R-COL0
- S31 pad 1: R-COL5 -> R-COL0
- S32 pad 1: R-COL5 -> R-COL0
- S33 pad 1: R-COL5 -> R-COL0
- S34 pad 1: R-COL5 -> R-COL0
- S35 pad 1: R-COL4 -> R-COL1
- S36 pad 1: R-COL4 -> R-COL1
- S37 pad 1: R-COL4 -> R-COL1
- S38 pad 1: R-COL4 -> R-COL1
- S39 pad 1: R-COL4 -> R-COL1
- S40 pad 1: R-COL3 -> R-COL2
- S41 pad 1: R-COL3 -> R-COL2
- S42 pad 1: R-COL3 -> R-COL2
- S43 pad 1: R-COL3 -> R-COL2
- S44 pad 1: R-COL3 -> R-COL2
- S45 pad 1: R-COL2 -> R-COL3
- S46 pad 1: R-COL2 -> R-COL3
- S47 pad 1: R-COL2 -> R-COL3
- S48 pad 1: R-COL2 -> R-COL3
- S49 pad 1: R-COL2 -> R-COL3
- S50 pad 1: R-COL1 -> R-COL4
- S51 pad 1: R-COL1 -> R-COL4
- S52 pad 1: R-COL1 -> R-COL4
- S53 pad 1: R-COL1 -> R-COL4
- S54 pad 1: R-COL1 -> R-COL4
- S55 pad 1: R-COL0 -> R-COL5
- S56 pad 1: R-COL0 -> R-COL5
- S57 pad 1: R-COL0 -> R-COL5
- S58 pad 1: R-COL0 -> R-COL5
- U1 pad 1: L-ENCODER-B0 -> L-RGB
- U1 pad 10: L-COL3 -> L-ROW2
- U1 pad 11: L-COL4 -> L-ROW3
- U1 pad 12: L-COL5 -> L-ROW4
- U1 pad 13: L-ROW4 -> L-COL4
- U1 pad 14: L-ROW3 -> L-COL3
- U1 pad 15: L-ROW2 -> L-COL2
- U1 pad 16: L-ROW1 -> L-COL1
- U1 pad 17: L-ROW0 -> L-COL0
- U1 pad 18: COMB -> L-COL5
- U1 pad 19: L-RGB -> L-ENCODER-A0
- U1 pad 2: L-ENCODER-A0 -> L-CS
- U1 pad 20: L-CS -> L-ENCODER-B0
- U1 pad 7: L-COL0 -> COMB
- U1 pad 8: L-COL1 -> L-ROW0
- U1 pad 9: L-COL2 -> L-ROW1
- U2 pad 1: unconnected-(U2-Pad1) -> R-RGB
- U2 pad 13: R-COL5 -> R-COL0
- U2 pad 14: R-COL4 -> R-COL1
- U2 pad 15: R-COL3 -> R-COL2
- U2 pad 16: R-COL2 -> R-COL3
- U2 pad 17: R-COL1 -> R-COL4
- U2 pad 18: R-COL0 -> R-COL5
- U2 pad 19: R-RGB -> R-RDY
- U2 pad 2: R-RDY -> R-CS
- U2 pad 20: R-CS -> unconnected-(U2-21-Pad20)
Routing:
- net COMB: track 0.00 -> 68.3 mm, vias 0 -> 2
- net +3V3: track 767.8 -> 826.5 mm
- net L-RGB: track 17.5 -> 38.6 mm
- net L-RST: track 46.8 -> 63.5 mm, vias 1 -> 0
- net L-COL0: track 230.6 -> 214.7 mm
- net Net-(SW1-B): track 48.7 -> 63.1 mm
- net GND: track 926.9 -> 940.9 mm, vias 30 -> 33
- net L-COL3: track 215.2 -> 201.9 mm
- net L-COL2: track 235.4 -> 223.8 mm
- net L-ROW1: track 169.2 -> 180.3 mm
- net L-COL4: track 196.3 -> 185.8 mm
- net L-BATTERY-POSITIVE: track 43.8 -> 54.3 mm
- net R-COL5: track 10.0 -> 20.1 mm
- net R-COL0: track 20.1 -> 10.0 mm
- net R-COL3: track 25.1 -> 15.1 mm
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